File: development/arena_12-12/ni/ni_arena_12-12_v0p1/layout_tool/modified_ni_arena_12-12.kicad_pcb (KiCad board)
At the start: 4 copper layers, 228.6 x 228.6 mm, 54 parts, among them J1 Barrel_Jack, J2 NI_TE_68pos, P1 CONN15, P10 CONN15, P11 CONN15, P12 CONN15, P2 CONN15, P3 CONN15, P4 CONN15, P5 CONN15, P6 CONN15, P7 CONN15, P8 CONN15, P9 CONN15, Q2 MOSFET_NCHAN, SW1 SW_SPDT, U1 TXB0108PW, U2 TXB0108PW, U3 TXB0108PW, U4 TXB0108PW, U5 TXB0108PW, U6 AP2112K-3.3

Commit message: Worked on layout for 12-12 ni arena with schmitt buffers.
Finished layout of components at base of panel columns.
Parts:
- removed the C1 at (120.6, 294.4)
- removed the C10 at (184.1, 294.4)
- removed the C2 at (108.1, 294.4)
- removed the C3 at (158.4, 294.4)
- removed the C4 at (146.2, 294.4)
- removed the C5 at (234.7, 294.4)
- removed the C6 at (222.2, 294.4)
- removed the C7 at (272.9, 294.7)
- removed the C8 at (260.4, 294.4)
- removed the C9 at (196.7, 294.3)
- added C100: 0.1uF, Capacitor_SMD:C_0402_1005Metric, F.Cu at (208.0, 268.0)
- added C101: 0.1uF, Capacitor_SMD:C_0402_1005Metric, F.Cu at (263.0, 216.7)
- added C102: 0.1uF, Capacitor_SMD:C_0402_1005Metric, F.Cu at (259.3, 223.2)
- added C103: 0.1uF, Capacitor_SMD:C_0402_1005Metric, F.Cu at (256.7, 227.7)
- added C104: 0.1uF, Capacitor_SMD:C_0402_1005Metric, F.Cu at (254.2, 232.0)
- added C105: 0.1uF, Capacitor_SMD:C_0402_1005Metric, F.Cu at (251.7, 236.4)
- added C106: 0.1uF, Capacitor_SMD:C_0402_1005Metric, F.Cu at (249.1, 240.8)
- added C107: 0.1uF, Capacitor_SMD:C_0402_1005Metric, F.Cu at (389.7, 90.0)
- added C108: 0.1uF, Capacitor_SMD:C_0402_1005Metric, F.Cu at (389.7, 92.0)
- added C109: 0.1uF, Capacitor_SMD:C_0402_1005Metric, F.Cu at (389.7, 94.0)
- added C110: 0.1uF, Capacitor_SMD:C_0402_1005Metric, F.Cu at (389.7, 96.0)
- added C111: 0.1uF, Capacitor_SMD:C_0402_1005Metric, F.Cu at (389.7, 97.9)
- added C112: 0.1uF, Capacitor_SMD:C_0402_1005Metric, F.Cu at (389.7, 99.9)
- added C113: 0.1uF, Capacitor_SMD:C_0402_1005Metric, F.Cu at (389.7, 101.9)
- added C114: 0.1uF, Capacitor_SMD:C_0402_1005Metric, F.Cu at (389.7, 103.8)
- added C115: 0.1uF, Capacitor_SMD:C_0402_1005Metric, F.Cu at (389.7, 105.8)
- added C116: 0.1uF, Capacitor_SMD:C_0402_1005Metric, F.Cu at (389.7, 107.8)
- added C117: 0.1uF, Capacitor_SMD:C_0402_1005Metric, F.Cu at (392.6, 90.0)
- added C118: 0.1uF, Capacitor_SMD:C_0402_1005Metric, F.Cu at (392.6, 92.0)
- added C119: 0.1uF, Capacitor_SMD:C_0402_1005Metric, F.Cu at (392.6, 94.0)
- added C120: 0.1uF, Capacitor_SMD:C_0402_1005Metric, F.Cu at (392.6, 96.0)
- added C121: 0.1uF, Capacitor_SMD:C_0402_1005Metric, F.Cu at (392.6, 97.9)
- added C122: 0.1uF, Capacitor_SMD:C_0402_1005Metric, F.Cu at (392.6, 99.9)
- added C123: 0.1uF, Capacitor_SMD:C_0402_1005Metric, F.Cu at (392.6, 101.9)
- added C124: 0.1uF, Capacitor_SMD:C_0402_1005Metric, F.Cu at (392.6, 103.8)
- added C125: 0.1uF, Capacitor_SMD:C_0402_1005Metric, F.Cu at (392.6, 105.8)
- added C126: 0.1uF, Capacitor_SMD:C_0402_1005Metric, F.Cu at (392.6, 107.8)
- added C127: 0.1uF, Capacitor_SMD:C_0402_1005Metric, F.Cu at (395.5, 90.0)
- added C128: 0.1uF, Capacitor_SMD:C_0402_1005Metric, F.Cu at (395.5, 92.0)
- added C129: 0.1uF, Capacitor_SMD:C_0402_1005Metric, F.Cu at (395.5, 94.0)
- added C13: 10uF, Capacitor_SMD:C_1206_3216Metric, F.Cu at (413.6, 78.8)
- added C130: 0.1uF, Capacitor_SMD:C_0402_1005Metric, F.Cu at (395.5, 96.0)
- added C131: 0.1uF, Capacitor_SMD:C_0402_1005Metric, F.Cu at (395.5, 97.9)
- added C132: 0.1uF, Capacitor_SMD:C_0402_1005Metric, F.Cu at (395.5, 99.9)
- added C133: 0.1uF, Capacitor_SMD:C_0402_1005Metric, F.Cu at (395.5, 101.9)
- added C134: 0.1uF, Capacitor_SMD:C_0402_1005Metric, F.Cu at (395.5, 103.8)
- added C135: 0.1uF, Capacitor_SMD:C_0402_1005Metric, F.Cu at (395.5, 105.8)
- added C136: 0.1uF, Capacitor_SMD:C_0402_1005Metric, F.Cu at (395.5, 107.8)
- added C137: 0.1uF, Capacitor_SMD:C_0402_1005Metric, F.Cu at (398.3, 90.0)
- added C138: 0.1uF, Capacitor_SMD:C_0402_1005Metric, F.Cu at (398.3, 92.0)
- added C139: 0.1uF, Capacitor_SMD:C_0402_1005Metric, F.Cu at (398.3, 94.0)
- added C14: 10uF, Capacitor_SMD:C_1206_3216Metric, F.Cu at (413.6, 82.2)
- added C140: 0.1uF, Capacitor_SMD:C_0402_1005Metric, F.Cu at (398.3, 96.0)
- added C15: 0.1uF, Capacitor_SMD:C_0402_1005Metric, F.Cu at (384.0, 90.0)
- added C16: 0.1uF, Capacitor_SMD:C_0402_1005Metric, F.Cu at (384.0, 92.0)
- added C17: 0.1uF, Capacitor_SMD:C_0402_1005Metric, F.Cu at (384.0, 94.0)
- added C18: 0.1uF, Capacitor_SMD:C_0402_1005Metric, F.Cu at (384.0, 96.0)
- added C19: 0.1uF, Capacitor_SMD:C_0402_1005Metric, F.Cu at (384.0, 97.9)
- added C20: 0.1uF, Capacitor_SMD:C_0402_1005Metric, F.Cu at (384.0, 99.9)
- added C21: 0.1uF, Capacitor_SMD:C_0402_1005Metric, F.Cu at (384.0, 101.9)
- added C22: 0.1uF, Capacitor_SMD:C_0402_1005Metric, F.Cu at (384.0, 103.8)
- added C25: 0.1uF, Capacitor_SMD:C_0402_1005Metric, F.Cu at (386.9, 90.0)
- added C26: 0.1uF, Capacitor_SMD:C_0402_1005Metric, F.Cu at (386.9, 92.0)
- added C27: 0.1uF, Capacitor_SMD:C_0402_1005Metric, F.Cu at (386.9, 94.0)
- added C28: 0.1uF, Capacitor_SMD:C_0402_1005Metric, F.Cu at (386.9, 96.0)
- added C29: 0.1uF, Capacitor_SMD:C_0402_1005Metric, F.Cu at (386.9, 97.9)
- added C30: 0.1uF, Capacitor_SMD:C_0402_1005Metric, F.Cu at (386.9, 99.9)
- added C31: 0.1uF, Capacitor_SMD:C_0402_1005Metric, F.Cu at (386.9, 101.9)
- added C32: 0.1uF, Capacitor_SMD:C_0402_1005Metric, F.Cu at (386.9, 103.8)
- added C33: 0.1uF, Capacitor_SMD:C_0402_1005Metric, F.Cu at (386.9, 105.8)
- added C34: 0.1uF, Capacitor_SMD:C_0402_1005Metric, F.Cu at (386.9, 107.8)
- added C35: 0.1uF, Capacitor_SMD:C_0402_1005Metric, F.Cu at (271.1, 168.9)
- added C36: 0.1uF, Capacitor_SMD:C_0402_1005Metric, F.Cu at (271.1, 176.4)
- added C37: 0.1uF, Capacitor_SMD:C_0402_1005Metric, F.Cu at (271.1, 181.5)
- added C38: 0.1uF, Capacitor_SMD:C_0402_1005Metric, F.Cu at (271.1, 186.6)
- added C39: 0.1uF, Capacitor_SMD:C_0402_1005Metric, F.Cu at (271.1, 191.6)
- added C40: 0.1uF, Capacitor_SMD:C_0402_1005Metric, F.Cu at (271.0, 196.7)
- added C41: 0.1uF, Capacitor_SMD:C_0402_1005Metric, F.Cu at (254.1, 123.4)
- added C42: 0.1uF, Capacitor_SMD:C_0402_1005Metric, F.Cu at (257.9, 129.9)
- added C43: 0.1uF, Capacitor_SMD:C_0402_1005Metric, F.Cu at (260.4, 134.4)
- added C44: 0.1uF, Capacitor_SMD:C_0402_1005Metric, F.Cu at (263.0, 138.8)
- added C45: 0.1uF, Capacitor_SMD:C_0402_1005Metric, F.Cu at (265.5, 143.2)
- added C46: 0.1uF, Capacitor_SMD:C_0402_1005Metric, F.Cu at (268.0, 147.6)
- added C47: 0.1uF, Capacitor_SMD:C_0402_1005Metric, F.Cu at (216.7, 92.6)
- added C48: 0.1uF, Capacitor_SMD:C_0402_1005Metric, F.Cu at (223.2, 96.3)
- added C49: 0.1uF, Capacitor_SMD:C_0402_1005Metric, F.Cu at (227.7, 98.9)
- added C50: 0.1uF, Capacitor_SMD:C_0402_1005Metric, F.Cu at (232.0, 101.4)
- added C51: 0.1uF, Capacitor_SMD:C_0402_1005Metric, F.Cu at (236.4, 103.9)
- added C52: 0.1uF, Capacitor_SMD:C_0402_1005Metric, F.Cu at (240.8, 106.5)
- added C53: 0.1uF, Capacitor_SMD:C_0402_1005Metric, F.Cu at (168.9, 84.5)
- added C54: 0.1uF, Capacitor_SMD:C_0402_1005Metric, F.Cu at (176.4, 84.5)
- added C55: 0.1uF, Capacitor_SMD:C_0402_1005Metric, F.Cu at (181.5, 84.5)
- added C56: 0.1uF, Capacitor_SMD:C_0402_1005Metric, F.Cu at (186.6, 84.5)
- added C57: 0.1uF, Capacitor_SMD:C_0402_1005Metric, F.Cu at (191.6, 84.5)
- added C58: 0.1uF, Capacitor_SMD:C_0402_1005Metric, F.Cu at (196.7, 84.6)
- added C59: 0.1uF, Capacitor_SMD:C_0402_1005Metric, F.Cu at (123.4, 101.5)
- added C60: 0.1uF, Capacitor_SMD:C_0402_1005Metric, F.Cu at (129.9, 97.7)
- added C61: 0.1uF, Capacitor_SMD:C_0402_1005Metric, F.Cu at (134.4, 95.2)
- added C62: 0.1uF, Capacitor_SMD:C_0402_1005Metric, F.Cu at (138.8, 92.6)
- added C63: 0.1uF, Capacitor_SMD:C_0402_1005Metric, F.Cu at (143.2, 90.1)
- added C64: 0.1uF, Capacitor_SMD:C_0402_1005Metric, F.Cu at (147.6, 87.6)
- added C65: 0.1uF, Capacitor_SMD:C_0402_1005Metric, F.Cu at (92.6, 138.9)
- added C66: 0.1uF, Capacitor_SMD:C_0402_1005Metric, F.Cu at (96.3, 132.4)
- added C67: 0.1uF, Capacitor_SMD:C_0402_1005Metric, F.Cu at (98.9, 127.9)
- added C68: 0.1uF, Capacitor_SMD:C_0402_1005Metric, F.Cu at (101.4, 123.6)
- added C69: 0.1uF, Capacitor_SMD:C_0402_1005Metric, F.Cu at (103.9, 119.2)
- added C70: 0.1uF, Capacitor_SMD:C_0402_1005Metric, F.Cu at (106.5, 114.8)
- added C71: 0.1uF, Capacitor_SMD:C_0402_1005Metric, F.Cu at (84.5, 186.7)
- added C72: 0.1uF, Capacitor_SMD:C_0402_1005Metric, F.Cu at (84.5, 179.2)
- added C73: 0.1uF, Capacitor_SMD:C_0402_1005Metric, F.Cu at (84.5, 174.1)
- added C74: 0.1uF, Capacitor_SMD:C_0402_1005Metric, F.Cu at (84.5, 169.0)
- added C75: 0.1uF, Capacitor_SMD:C_0402_1005Metric, F.Cu at (84.5, 164.0)
- added C76: 0.1uF, Capacitor_SMD:C_0402_1005Metric, F.Cu at (84.6, 158.9)
- added C77: 0.1uF, Capacitor_SMD:C_0402_1005Metric, F.Cu at (101.5, 232.2)
- added C78: 0.1uF, Capacitor_SMD:C_0402_1005Metric, F.Cu at (97.7, 225.7)
- added C79: 0.1uF, Capacitor_SMD:C_0402_1005Metric, F.Cu at (95.2, 221.2)
- added C80: 0.1uF, Capacitor_SMD:C_0402_1005Metric, F.Cu at (92.6, 216.8)
- added C81: 0.1uF, Capacitor_SMD:C_0402_1005Metric, F.Cu at (90.1, 212.4)
- added C82: 0.1uF, Capacitor_SMD:C_0402_1005Metric, F.Cu at (87.6, 208.0)
- added C83: 0.1uF, Capacitor_SMD:C_0402_1005Metric, F.Cu at (138.9, 263.0)
- added C84: 0.1uF, Capacitor_SMD:C_0402_1005Metric, F.Cu at (132.4, 259.3)
- added C85: 0.1uF, Capacitor_SMD:C_0402_1005Metric, F.Cu at (127.9, 256.7)
- added C86: 0.1uF, Capacitor_SMD:C_0402_1005Metric, F.Cu at (123.6, 254.2)
- added C87: 0.1uF, Capacitor_SMD:C_0402_1005Metric, F.Cu at (119.2, 251.7)
- added C88: 0.1uF, Capacitor_SMD:C_0402_1005Metric, F.Cu at (114.8, 249.1)
- added C89: 0.1uF, Capacitor_SMD:C_0402_1005Metric, F.Cu at (186.7, 271.1)
- added C90: 0.1uF, Capacitor_SMD:C_0402_1005Metric, F.Cu at (179.2, 271.1)
- added C91: 0.1uF, Capacitor_SMD:C_0402_1005Metric, F.Cu at (174.1, 271.1)
- added C92: 0.1uF, Capacitor_SMD:C_0402_1005Metric, F.Cu at (169.0, 271.1)
- added C93: 0.1uF, Capacitor_SMD:C_0402_1005Metric, F.Cu at (164.0, 271.1)
- added C94: 0.1uF, Capacitor_SMD:C_0402_1005Metric, F.Cu at (158.9, 271.0)
- added C95: 0.1uF, Capacitor_SMD:C_0402_1005Metric, F.Cu at (232.2, 254.1)
- added C96: 0.1uF, Capacitor_SMD:C_0402_1005Metric, F.Cu at (225.7, 257.9)
- added C97: 0.1uF, Capacitor_SMD:C_0402_1005Metric, F.Cu at (221.2, 260.4)
- added C98: 0.1uF, Capacitor_SMD:C_0402_1005Metric, F.Cu at (216.8, 263.0)
- added C99: 0.1uF, Capacitor_SMD:C_0402_1005Metric, F.Cu at (212.4, 265.5)
- added J3: Barrel_Jack, arena_custom:DCJACK_2PIN_HIGHCURRENT, F.Cu at (95.0, 63.5)
- added R10: 33, Resistor_SMD:R_0402_1005Metric, F.Cu at (415.1, 62.2)
- added R100: 33, Resistor_SMD:R_0402_1005Metric, F.Cu at (395.6, 82.1)
- added R101: 33, Resistor_SMD:R_0402_1005Metric, F.Cu at (395.6, 84.1)
- added R102: 33, Resistor_SMD:R_0402_1005Metric, F.Cu at (395.6, 86.1)
- added R103: 33, Resistor_SMD:R_0402_1005Metric, F.Cu at (395.6, 88.1)
- added R104: 33, Resistor_SMD:R_0402_1005Metric, F.Cu at (398.6, 60.2)
- added R105: 33, Resistor_SMD:R_0402_1005Metric, F.Cu at (398.6, 62.2)
- added R106: 33, Resistor_SMD:R_0402_1005Metric, F.Cu at (398.6, 64.2)
- added R107: 33, Resistor_SMD:R_0402_1005Metric, F.Cu at (398.6, 66.2)
- added R108: 33, Resistor_SMD:R_0402_1005Metric, F.Cu at (398.6, 68.2)
- added R109: 33, Resistor_SMD:R_0402_1005Metric, F.Cu at (398.6, 70.2)
- added R11: 33, Resistor_SMD:R_0402_1005Metric, F.Cu at (415.1, 64.2)
- added R110: 33, Resistor_SMD:R_0402_1005Metric, F.Cu at (398.6, 72.1)
- added R111: 33, Resistor_SMD:R_0402_1005Metric, F.Cu at (398.6, 74.1)
- added R112: 33, Resistor_SMD:R_0402_1005Metric, F.Cu at (398.6, 76.1)
- added R113: 33, Resistor_SMD:R_0402_1005Metric, F.Cu at (398.6, 78.1)
- added R114: 33, Resistor_SMD:R_0402_1005Metric, F.Cu at (398.6, 80.1)
- added R115: 33, Resistor_SMD:R_0402_1005Metric, F.Cu at (398.6, 82.1)
- added R116: 33, Resistor_SMD:R_0402_1005Metric, F.Cu at (398.6, 84.1)
- added R117: 33, Resistor_SMD:R_0402_1005Metric, F.Cu at (398.6, 86.1)
- added R118: 33, Resistor_SMD:R_0402_1005Metric, F.Cu at (398.6, 88.1)
- added R119: 33, Resistor_SMD:R_0402_1005Metric, F.Cu at (401.5, 60.2)
- added R12: 33, Resistor_SMD:R_0402_1005Metric, F.Cu at (415.1, 66.2)
- added R120: 33, Resistor_SMD:R_0402_1005Metric, F.Cu at (401.5, 62.2)
- added R121: 33, Resistor_SMD:R_0402_1005Metric, F.Cu at (401.5, 64.2)
- added R122: 33, Resistor_SMD:R_0402_1005Metric, F.Cu at (401.5, 66.2)
- added R123: 33, Resistor_SMD:R_0402_1005Metric, F.Cu at (401.5, 68.2)
- added R124: 33, Resistor_SMD:R_0402_1005Metric, F.Cu at (401.5, 70.2)
- added R125: 33, Resistor_SMD:R_0402_1005Metric, F.Cu at (401.5, 72.1)
- added R126: 33, Resistor_SMD:R_0402_1005Metric, F.Cu at (401.5, 74.1)
- added R127: 33, Resistor_SMD:R_0402_1005Metric, F.Cu at (401.5, 76.1)
- added R128: 33, Resistor_SMD:R_0402_1005Metric, F.Cu at (401.5, 78.1)
- added R129: 33, Resistor_SMD:R_0402_1005Metric, F.Cu at (401.5, 80.1)
- added R13: 33, Resistor_SMD:R_0402_1005Metric, F.Cu at (415.1, 68.2)
- added R130: 33, Resistor_SMD:R_0402_1005Metric, F.Cu at (401.5, 82.1)
- added R131: 33, Resistor_SMD:R_0402_1005Metric, F.Cu at (401.5, 84.1)
- added R132: 33, Resistor_SMD:R_0402_1005Metric, F.Cu at (401.5, 86.1)
- added R133: 33, Resistor_SMD:R_0402_1005Metric, F.Cu at (401.5, 88.1)
- added R134: 33, Resistor_SMD:R_0402_1005Metric, F.Cu at (404.4, 60.2)
- added R135: 33, Resistor_SMD:R_0402_1005Metric, F.Cu at (404.4, 62.2)
- added R136: 33, Resistor_SMD:R_0402_1005Metric, F.Cu at (404.4, 64.2)
- added R137: 33, Resistor_SMD:R_0402_1005Metric, F.Cu at (404.4, 66.2)
- added R138: 33, Resistor_SMD:R_0402_1005Metric, F.Cu at (404.4, 68.2)
- added R139: 33, Resistor_SMD:R_0402_1005Metric, F.Cu at (404.4, 70.2)
- added R14: 33, Resistor_SMD:R_0402_1005Metric, F.Cu at (415.1, 70.2)
- added R140: 33, Resistor_SMD:R_0402_1005Metric, F.Cu at (404.4, 72.1)
- added R141: 33, Resistor_SMD:R_0402_1005Metric, F.Cu at (404.4, 74.1)
- added R142: 33, Resistor_SMD:R_0402_1005Metric, F.Cu at (404.4, 76.1)
- added R143: 33, Resistor_SMD:R_0402_1005Metric, F.Cu at (404.4, 78.1)
- added R144: 33, Resistor_SMD:R_0402_1005Metric, F.Cu at (404.4, 80.1)
- added R145: 33, Resistor_SMD:R_0402_1005Metric, F.Cu at (404.4, 82.1)
- added R146: 33, Resistor_SMD:R_0402_1005Metric, F.Cu at (404.4, 84.1)
- added R147: 33, Resistor_SMD:R_0402_1005Metric, F.Cu at (404.4, 86.1)
- added R148: 33, Resistor_SMD:R_0402_1005Metric, F.Cu at (404.4, 88.1)
- added R149: 33, Resistor_SMD:R_0402_1005Metric, F.Cu at (407.3, 60.2)
- added R15: 33, Resistor_SMD:R_0402_1005Metric, F.Cu at (415.1, 72.1)
- added R150: 33, Resistor_SMD:R_0402_1005Metric, F.Cu at (407.3, 62.2)
- added R151: 33, Resistor_SMD:R_0402_1005Metric, F.Cu at (407.3, 64.2)
- added R152: 33, Resistor_SMD:R_0402_1005Metric, F.Cu at (407.3, 66.2)
- added R153: 33, Resistor_SMD:R_0402_1005Metric, F.Cu at (407.3, 68.2)
- added R154: 33, Resistor_SMD:R_0402_1005Metric, F.Cu at (407.3, 70.2)
- added R155: 33, Resistor_SMD:R_0402_1005Metric, F.Cu at (407.3, 72.1)
- added R156: 33, Resistor_SMD:R_0402_1005Metric, F.Cu at (407.3, 74.1)
- added R157: 33, Resistor_SMD:R_0402_1005Metric, F.Cu at (407.3, 76.1)
- added R158: 33, Resistor_SMD:R_0402_1005Metric, F.Cu at (407.3, 78.1)
- added R159: 33, Resistor_SMD:R_0402_1005Metric, F.Cu at (407.3, 80.1)
- added R16: 33, Resistor_SMD:R_0402_1005Metric, F.Cu at (415.1, 74.1)
- added R160: 33, Resistor_SMD:R_0402_1005Metric, F.Cu at (407.3, 82.1)
- added R161: 33, Resistor_SMD:R_0402_1005Metric, F.Cu at (407.3, 84.1)
- added R162: 33, Resistor_SMD:R_0402_1005Metric, F.Cu at (407.3, 86.1)
- added R163: 33, Resistor_SMD:R_0402_1005Metric, F.Cu at (271.1, 167.8)
- added R164: 33, Resistor_SMD:R_0402_1005Metric, F.Cu at (271.1, 169.9)
- added R165: 33, Resistor_SMD:R_0402_1005Metric, F.Cu at (271.1, 172.7)
- added R166: 33, Resistor_SMD:R_0402_1005Metric, F.Cu at (271.1, 175.2)
- added R167: 33, Resistor_SMD:R_0402_1005Metric, F.Cu at (271.1, 177.5)
- added R168: 33, Resistor_SMD:R_0402_1005Metric, F.Cu at (271.1, 180.3)
- added R169: 33, Resistor_SMD:R_0402_1005Metric, F.Cu at (271.1, 182.7)
- added R17: 33, Resistor_SMD:R_0402_1005Metric, F.Cu at (418.0, 60.2)
- added R170: 33, Resistor_SMD:R_0402_1005Metric, F.Cu at (271.1, 185.4)
- added R171: 33, Resistor_SMD:R_0402_1005Metric, F.Cu at (271.1, 187.7)
- added R172: 33, Resistor_SMD:R_0402_1005Metric, F.Cu at (271.1, 190.5)
- added R173: 33, Resistor_SMD:R_0402_1005Metric, F.Cu at (271.1, 192.8)
- added R174: 33, Resistor_SMD:R_0402_1005Metric, F.Cu at (271.1, 195.6)
- added R175: 33, Resistor_SMD:R_0402_1005Metric, F.Cu at (253.6, 122.5)
- added R176: 33, Resistor_SMD:R_0402_1005Metric, F.Cu at (254.7, 124.4)
- added R177: 33, Resistor_SMD:R_0402_1005Metric, F.Cu at (256.1, 126.7)
- added R178: 33, Resistor_SMD:R_0402_1005Metric, F.Cu at (257.3, 129.0)
- added R179: 33, Resistor_SMD:R_0402_1005Metric, F.Cu at (258.4, 130.9)
- added R18: 33, Resistor_SMD:R_0402_1005Metric, F.Cu at (418.0, 62.2)
- added R180: 33, Resistor_SMD:R_0402_1005Metric, F.Cu at (259.8, 133.4)
- added R181: 33, Resistor_SMD:R_0402_1005Metric, F.Cu at (261.0, 135.4)
- added R182: 33, Resistor_SMD:R_0402_1005Metric, F.Cu at (262.4, 137.8)
- added R183: 33, Resistor_SMD:R_0402_1005Metric, F.Cu at (263.5, 139.8)
- added R184: 33, Resistor_SMD:R_0402_1005Metric, F.Cu at (264.9, 142.2)
- added R185: 33, Resistor_SMD:R_0402_1005Metric, F.Cu at (266.1, 144.1)
- added R186: 33, Resistor_SMD:R_0402_1005Metric, F.Cu at (267.5, 146.6)
- added R187: 33, Resistor_SMD:R_0402_1005Metric, F.Cu at (215.8, 92.0)
- added R188: 33, Resistor_SMD:R_0402_1005Metric, F.Cu at (217.6, 93.1)
- added R189: 33, Resistor_SMD:R_0402_1005Metric, F.Cu at (220.1, 94.5)
- added R19: 33, Resistor_SMD:R_0402_1005Metric, F.Cu at (418.0, 64.2)
- added R190: 33, Resistor_SMD:R_0402_1005Metric, F.Cu at (222.2, 95.8)
- added R191: 33, Resistor_SMD:R_0402_1005Metric, F.Cu at (224.2, 96.9)
- added R192: 33, Resistor_SMD:R_0402_1005Metric, F.Cu at (226.6, 98.3)
- added R193: 33, Resistor_SMD:R_0402_1005Metric, F.Cu at (228.6, 99.4)
- added R194: 33, Resistor_SMD:R_0402_1005Metric, F.Cu at (231.0, 100.8)
- added R195: 33, Resistor_SMD:R_0402_1005Metric, F.Cu at (233.0, 102.0)
- added R196: 33, Resistor_SMD:R_0402_1005Metric, F.Cu at (235.4, 103.4)
- added R197: 33, Resistor_SMD:R_0402_1005Metric, F.Cu at (237.4, 104.5)
- added R198: 33, Resistor_SMD:R_0402_1005Metric, F.Cu at (239.8, 105.9)
- added R199: 33, Resistor_SMD:R_0402_1005Metric, F.Cu at (167.8, 84.5)
- added R20: 33, Resistor_SMD:R_0402_1005Metric, F.Cu at (418.0, 66.2)
- added R200: 33, Resistor_SMD:R_0402_1005Metric, F.Cu at (169.9, 84.5)
- added R201: 33, Resistor_SMD:R_0402_1005Metric, F.Cu at (172.7, 84.5)
- added R202: 33, Resistor_SMD:R_0402_1005Metric, F.Cu at (175.2, 84.5)
- added R203: 33, Resistor_SMD:R_0402_1005Metric, F.Cu at (177.5, 84.5)
- added R204: 33, Resistor_SMD:R_0402_1005Metric, F.Cu at (180.3, 84.5)
- added R205: 33, Resistor_SMD:R_0402_1005Metric, F.Cu at (182.7, 84.5)
- added R206: 33, Resistor_SMD:R_0402_1005Metric, F.Cu at (185.4, 84.5)
- added R207: 33, Resistor_SMD:R_0402_1005Metric, F.Cu at (187.7, 84.5)
- added R208: 33, Resistor_SMD:R_0402_1005Metric, F.Cu at (190.5, 84.5)
- added R209: 33, Resistor_SMD:R_0402_1005Metric, F.Cu at (192.8, 84.5)
- added R21: 33, Resistor_SMD:R_0402_1005Metric, F.Cu at (418.0, 68.2)
- added R210: 33, Resistor_SMD:R_0402_1005Metric, F.Cu at (195.6, 84.5)
- added R211: 33, Resistor_SMD:R_0402_1005Metric, F.Cu at (122.5, 102.0)
- added R212: 33, Resistor_SMD:R_0402_1005Metric, F.Cu at (124.4, 100.9)
- added R213: 33, Resistor_SMD:R_0402_1005Metric, F.Cu at (126.7, 99.5)
- added R214: 33, Resistor_SMD:R_0402_1005Metric, F.Cu at (129.0, 98.3)
- added R215: 33, Resistor_SMD:R_0402_1005Metric, F.Cu at (130.9, 97.2)
- added R216: 33, Resistor_SMD:R_0402_1005Metric, F.Cu at (133.4, 95.8)
- added R217: 33, Resistor_SMD:R_0402_1005Metric, F.Cu at (135.4, 94.6)
- added R218: 33, Resistor_SMD:R_0402_1005Metric, F.Cu at (137.8, 93.2)
- added R219: 33, Resistor_SMD:R_0402_1005Metric, F.Cu at (139.8, 92.1)
- added R22: 33, Resistor_SMD:R_0402_1005Metric, F.Cu at (418.0, 70.2)
- added R220: 33, Resistor_SMD:R_0402_1005Metric, F.Cu at (142.2, 90.7)
- added R221: 33, Resistor_SMD:R_0402_1005Metric, F.Cu at (144.1, 89.5)
- added R222: 33, Resistor_SMD:R_0402_1005Metric, F.Cu at (146.6, 88.1)
- added R223: 33, Resistor_SMD:R_0402_1005Metric, F.Cu at (92.0, 139.8)
- added R224: 33, Resistor_SMD:R_0402_1005Metric, F.Cu at (93.1, 138.0)
- added R225: 33, Resistor_SMD:R_0402_1005Metric, F.Cu at (94.5, 135.5)
- added R226: 33, Resistor_SMD:R_0402_1005Metric, F.Cu at (95.8, 133.4)
- added R227: 33, Resistor_SMD:R_0402_1005Metric, F.Cu at (96.9, 131.4)
- added R228: 33, Resistor_SMD:R_0402_1005Metric, F.Cu at (98.3, 129.0)
- added R229: 33, Resistor_SMD:R_0402_1005Metric, F.Cu at (99.4, 127.0)
- added R23: 33, Resistor_SMD:R_0402_1005Metric, F.Cu at (418.0, 72.1)
- added R230: 33, Resistor_SMD:R_0402_1005Metric, F.Cu at (100.8, 124.6)
- added R231: 33, Resistor_SMD:R_0402_1005Metric, F.Cu at (102.0, 122.6)
- added R232: 33, Resistor_SMD:R_0402_1005Metric, F.Cu at (103.4, 120.2)
- added R233: 33, Resistor_SMD:R_0402_1005Metric, F.Cu at (104.5, 118.2)
- added R234: 33, Resistor_SMD:R_0402_1005Metric, F.Cu at (105.9, 115.8)
- added R235: 33, Resistor_SMD:R_0402_1005Metric, F.Cu at (84.5, 187.8)
- added R236: 33, Resistor_SMD:R_0402_1005Metric, F.Cu at (84.5, 185.7)
- added R237: 33, Resistor_SMD:R_0402_1005Metric, F.Cu at (84.5, 182.9)
- added R238: 33, Resistor_SMD:R_0402_1005Metric, F.Cu at (84.5, 180.3)
- added R239: 33, Resistor_SMD:R_0402_1005Metric, F.Cu at (84.5, 178.1)
- added R24: 33, Resistor_SMD:R_0402_1005Metric, F.Cu at (418.0, 74.1)
- added R240: 33, Resistor_SMD:R_0402_1005Metric, F.Cu at (84.5, 175.3)
- added R241: 33, Resistor_SMD:R_0402_1005Metric, F.Cu at (84.5, 172.9)
- added R242: 33, Resistor_SMD:R_0402_1005Metric, F.Cu at (84.5, 170.2)
- added R243: 33, Resistor_SMD:R_0402_1005Metric, F.Cu at (84.5, 167.9)
- added R244: 33, Resistor_SMD:R_0402_1005Metric, F.Cu at (84.5, 165.1)
- added R245: 33, Resistor_SMD:R_0402_1005Metric, F.Cu at (84.5, 162.8)
- added R246: 33, Resistor_SMD:R_0402_1005Metric, F.Cu at (84.5, 160.0)
- added R247: 33, Resistor_SMD:R_0402_1005Metric, F.Cu at (102.0, 233.1)
- added R248: 33, Resistor_SMD:R_0402_1005Metric, F.Cu at (100.9, 231.2)
- added R249: 33, Resistor_SMD:R_0402_1005Metric, F.Cu at (99.5, 228.9)
- added R25: 33, Resistor_SMD:R_0402_1005Metric, F.Cu at (420.9, 60.2)
- added R250: 33, Resistor_SMD:R_0402_1005Metric, F.Cu at (98.3, 226.6)
- added R251: 33, Resistor_SMD:R_0402_1005Metric, F.Cu at (97.2, 224.7)
- added R252: 33, Resistor_SMD:R_0402_1005Metric, F.Cu at (95.8, 222.2)
- added R253: 33, Resistor_SMD:R_0402_1005Metric, F.Cu at (94.6, 220.2)
- added R254: 33, Resistor_SMD:R_0402_1005Metric, F.Cu at (93.2, 217.8)
- added R255: 33, Resistor_SMD:R_0402_1005Metric, F.Cu at (92.1, 215.8)
- added R256: 33, Resistor_SMD:R_0402_1005Metric, F.Cu at (90.7, 213.4)
- added R257: 33, Resistor_SMD:R_0402_1005Metric, F.Cu at (89.5, 211.5)
- added R258: 33, Resistor_SMD:R_0402_1005Metric, F.Cu at (88.1, 209.0)
- added R259: 33, Resistor_SMD:R_0402_1005Metric, F.Cu at (139.8, 263.6)
- added R26: 33, Resistor_SMD:R_0402_1005Metric, F.Cu at (420.9, 62.2)
- added R260: 33, Resistor_SMD:R_0402_1005Metric, F.Cu at (138.0, 262.5)
- added R261: 33, Resistor_SMD:R_0402_1005Metric, F.Cu at (135.5, 261.1)
- added R262: 33, Resistor_SMD:R_0402_1005Metric, F.Cu at (133.4, 259.8)
- added R263: 33, Resistor_SMD:R_0402_1005Metric, F.Cu at (131.4, 258.7)
- added R264: 33, Resistor_SMD:R_0402_1005Metric, F.Cu at (129.0, 257.3)
- added R265: 33, Resistor_SMD:R_0402_1005Metric, F.Cu at (127.0, 256.2)
- added R266: 33, Resistor_SMD:R_0402_1005Metric, F.Cu at (124.6, 254.8)
- added R267: 33, Resistor_SMD:R_0402_1005Metric, F.Cu at (122.6, 253.6)
- added R268: 33, Resistor_SMD:R_0402_1005Metric, F.Cu at (120.2, 252.2)
- added R269: 33, Resistor_SMD:R_0402_1005Metric, F.Cu at (118.2, 251.1)
- added R27: 33, Resistor_SMD:R_0402_1005Metric, F.Cu at (420.9, 64.2)
- added R270: 33, Resistor_SMD:R_0402_1005Metric, F.Cu at (115.8, 249.7)
- added R271: 33, Resistor_SMD:R_0402_1005Metric, F.Cu at (187.8, 271.1)
- added R272: 33, Resistor_SMD:R_0402_1005Metric, F.Cu at (185.7, 271.1)
- added R273: 33, Resistor_SMD:R_0402_1005Metric, F.Cu at (182.9, 271.1)
- added R274: 33, Resistor_SMD:R_0402_1005Metric, F.Cu at (180.3, 271.1)
- added R275: 33, Resistor_SMD:R_0402_1005Metric, F.Cu at (178.1, 271.1)
- added R276: 33, Resistor_SMD:R_0402_1005Metric, F.Cu at (175.3, 271.1)
- added R277: 33, Resistor_SMD:R_0402_1005Metric, F.Cu at (172.9, 271.1)
- added R278: 33, Resistor_SMD:R_0402_1005Metric, F.Cu at (170.2, 271.1)
- added R279: 33, Resistor_SMD:R_0402_1005Metric, F.Cu at (167.9, 271.1)
- added R28: 33, Resistor_SMD:R_0402_1005Metric, F.Cu at (420.9, 66.2)
- added R280: 33, Resistor_SMD:R_0402_1005Metric, F.Cu at (165.1, 271.1)
- added R281: 33, Resistor_SMD:R_0402_1005Metric, F.Cu at (162.8, 271.1)
- added R282: 33, Resistor_SMD:R_0402_1005Metric, F.Cu at (160.0, 271.1)
- added R283: 33, Resistor_SMD:R_0402_1005Metric, F.Cu at (233.1, 253.6)
- added R284: 33, Resistor_SMD:R_0402_1005Metric, F.Cu at (231.2, 254.7)
- added R285: 33, Resistor_SMD:R_0402_1005Metric, F.Cu at (228.9, 256.1)
- added R286: 33, Resistor_SMD:R_0402_1005Metric, F.Cu at (226.6, 257.3)
- added R287: 33, Resistor_SMD:R_0402_1005Metric, F.Cu at (224.7, 258.4)
- added R288: 33, Resistor_SMD:R_0402_1005Metric, F.Cu at (222.2, 259.8)
- added R289: 33, Resistor_SMD:R_0402_1005Metric, F.Cu at (220.2, 261.0)
- added R29: 33, Resistor_SMD:R_0402_1005Metric, F.Cu at (384.0, 60.2)
- added R290: 33, Resistor_SMD:R_0402_1005Metric, F.Cu at (217.8, 262.4)
- added R291: 33, Resistor_SMD:R_0402_1005Metric, F.Cu at (215.8, 263.5)
- added R292: 33, Resistor_SMD:R_0402_1005Metric, F.Cu at (213.4, 264.9)
- added R293: 33, Resistor_SMD:R_0402_1005Metric, F.Cu at (211.5, 266.1)
- added R294: 33, Resistor_SMD:R_0402_1005Metric, F.Cu at (209.0, 267.5)
- added R295: 33, Resistor_SMD:R_0402_1005Metric, F.Cu at (263.6, 215.8)
- added R296: 33, Resistor_SMD:R_0402_1005Metric, F.Cu at (262.5, 217.6)
- added R297: 33, Resistor_SMD:R_0402_1005Metric, F.Cu at (261.1, 220.1)
- added R298: 33, Resistor_SMD:R_0402_1005Metric, F.Cu at (259.8, 222.2)
- added R299: 33, Resistor_SMD:R_0402_1005Metric, F.Cu at (258.7, 224.2)
- added R3: 33, Resistor_SMD:R_0402_1005Metric, F.Cu at (412.2, 64.2)
- added R30: 33, Resistor_SMD:R_0402_1005Metric, F.Cu at (384.0, 62.2)
- added R300: 33, Resistor_SMD:R_0402_1005Metric, F.Cu at (257.3, 226.6)
- added R301: 33, Resistor_SMD:R_0402_1005Metric, F.Cu at (256.2, 228.6)
- added R302: 33, Resistor_SMD:R_0402_1005Metric, F.Cu at (254.8, 231.0)
- added R303: 33, Resistor_SMD:R_0402_1005Metric, F.Cu at (253.6, 233.0)
- added R304: 33, Resistor_SMD:R_0402_1005Metric, F.Cu at (252.2, 235.4)
- added R305: 33, Resistor_SMD:R_0402_1005Metric, F.Cu at (251.1, 237.4)
- added R306: 33, Resistor_SMD:R_0402_1005Metric, F.Cu at (249.7, 239.8)
- added R307: 20k, Resistor_SMD:R_0402_1005Metric, F.Cu at (417.1, 30.6)
- added R308: 200, Resistor_SMD:R_0402_1005Metric, F.Cu at (417.1, 32.5)
- added R31: 33, Resistor_SMD:R_0402_1005Metric, F.Cu at (384.0, 64.2)
- added R32: 33, Resistor_SMD:R_0402_1005Metric, F.Cu at (384.0, 66.2)
- added R33: 33, Resistor_SMD:R_0402_1005Metric, F.Cu at (384.0, 68.2)
- added R34: 33, Resistor_SMD:R_0402_1005Metric, F.Cu at (384.0, 70.2)
- added R35: 33, Resistor_SMD:R_0402_1005Metric, F.Cu at (384.0, 72.1)
- added R36: 33, Resistor_SMD:R_0402_1005Metric, F.Cu at (384.0, 74.1)
- added R37: 33, Resistor_SMD:R_0402_1005Metric, F.Cu at (384.0, 76.1)
- added R38: 33, Resistor_SMD:R_0402_1005Metric, F.Cu at (384.0, 78.1)
- added R39: 33, Resistor_SMD:R_0402_1005Metric, F.Cu at (384.0, 80.1)
- added R4: 33, Resistor_SMD:R_0402_1005Metric, F.Cu at (412.2, 66.2)
- added R40: 33, Resistor_SMD:R_0402_1005Metric, F.Cu at (384.0, 82.1)
- added R41: 33, Resistor_SMD:R_0402_1005Metric, F.Cu at (384.0, 84.1)
- added R42: 33, Resistor_SMD:R_0402_1005Metric, F.Cu at (384.0, 86.1)
- added R43: 33, Resistor_SMD:R_0402_1005Metric, F.Cu at (384.0, 88.1)
- added R44: 33, Resistor_SMD:R_0402_1005Metric, F.Cu at (386.9, 60.2)
- added R45: 33, Resistor_SMD:R_0402_1005Metric, F.Cu at (386.9, 62.2)
- added R46: 33, Resistor_SMD:R_0402_1005Metric, F.Cu at (386.9, 64.2)
- added R47: 33, Resistor_SMD:R_0402_1005Metric, F.Cu at (386.9, 66.2)
- added R48: 33, Resistor_SMD:R_0402_1005Metric, F.Cu at (386.9, 68.2)
- added R49: 33, Resistor_SMD:R_0402_1005Metric, F.Cu at (386.9, 70.2)
- added R5: 33, Resistor_SMD:R_0402_1005Metric, F.Cu at (412.2, 68.2)
- added R50: 33, Resistor_SMD:R_0402_1005Metric, F.Cu at (386.9, 72.1)
- added R51: 33, Resistor_SMD:R_0402_1005Metric, F.Cu at (386.9, 74.1)
- added R52: 33, Resistor_SMD:R_0402_1005Metric, F.Cu at (386.9, 76.1)
- added R53: 33, Resistor_SMD:R_0402_1005Metric, F.Cu at (386.9, 78.1)
- added R54: 33, Resistor_SMD:R_0402_1005Metric, F.Cu at (386.9, 80.1)
- added R55: 33, Resistor_SMD:R_0402_1005Metric, F.Cu at (386.9, 82.1)
- added R56: 33, Resistor_SMD:R_0402_1005Metric, F.Cu at (386.9, 84.1)
- added R57: 33, Resistor_SMD:R_0402_1005Metric, F.Cu at (386.9, 86.1)
- added R58: 33, Resistor_SMD:R_0402_1005Metric, F.Cu at (386.9, 88.1)
- added R59: 33, Resistor_SMD:R_0402_1005Metric, F.Cu at (389.8, 60.2)
- added R6: 33, Resistor_SMD:R_0402_1005Metric, F.Cu at (412.2, 70.2)
- added R60: 33, Resistor_SMD:R_0402_1005Metric, F.Cu at (389.8, 62.2)
- added R61: 33, Resistor_SMD:R_0402_1005Metric, F.Cu at (389.8, 64.2)
- added R62: 33, Resistor_SMD:R_0402_1005Metric, F.Cu at (389.8, 66.2)
- added R63: 33, Resistor_SMD:R_0402_1005Metric, F.Cu at (389.8, 68.2)
- added R64: 33, Resistor_SMD:R_0402_1005Metric, F.Cu at (389.8, 70.2)
- added R65: 33, Resistor_SMD:R_0402_1005Metric, F.Cu at (389.8, 72.1)
- added R66: 33, Resistor_SMD:R_0402_1005Metric, F.Cu at (389.8, 74.1)
- added R67: 33, Resistor_SMD:R_0402_1005Metric, F.Cu at (389.8, 76.1)
- added R68: 33, Resistor_SMD:R_0402_1005Metric, F.Cu at (389.8, 78.1)
- added R69: 33, Resistor_SMD:R_0402_1005Metric, F.Cu at (389.8, 80.1)
- added R7: 33, Resistor_SMD:R_0402_1005Metric, F.Cu at (412.2, 72.1)
- added R70: 33, Resistor_SMD:R_0402_1005Metric, F.Cu at (389.8, 82.1)
- added R71: 33, Resistor_SMD:R_0402_1005Metric, F.Cu at (389.8, 84.1)
- added R72: 33, Resistor_SMD:R_0402_1005Metric, F.Cu at (389.8, 86.1)
- added R73: 33, Resistor_SMD:R_0402_1005Metric, F.Cu at (389.8, 88.1)
- added R74: 33, Resistor_SMD:R_0402_1005Metric, F.Cu at (392.7, 60.2)
- added R75: 33, Resistor_SMD:R_0402_1005Metric, F.Cu at (392.7, 62.2)
- added R76: 33, Resistor_SMD:R_0402_1005Metric, F.Cu at (392.7, 64.2)
- added R77: 33, Resistor_SMD:R_0402_1005Metric, F.Cu at (392.7, 66.2)
- added R78: 33, Resistor_SMD:R_0402_1005Metric, F.Cu at (392.7, 68.2)
- added R79: 33, Resistor_SMD:R_0402_1005Metric, F.Cu at (392.7, 70.2)
- added R8: 33, Resistor_SMD:R_0402_1005Metric, F.Cu at (412.2, 74.1)
- added R80: 33, Resistor_SMD:R_0402_1005Metric, F.Cu at (392.7, 72.1)
- added R81: 33, Resistor_SMD:R_0402_1005Metric, F.Cu at (392.7, 74.1)
- added R82: 33, Resistor_SMD:R_0402_1005Metric, F.Cu at (392.7, 76.1)
- added R83: 33, Resistor_SMD:R_0402_1005Metric, F.Cu at (392.7, 78.1)
- added R84: 33, Resistor_SMD:R_0402_1005Metric, F.Cu at (392.7, 80.1)
- added R85: 33, Resistor_SMD:R_0402_1005Metric, F.Cu at (392.7, 82.1)
- added R86: 33, Resistor_SMD:R_0402_1005Metric, F.Cu at (392.7, 84.1)
- added R87: 33, Resistor_SMD:R_0402_1005Metric, F.Cu at (392.7, 86.1)
- added R88: 33, Resistor_SMD:R_0402_1005Metric, F.Cu at (392.7, 88.1)
- added R89: 33, Resistor_SMD:R_0402_1005Metric, F.Cu at (395.6, 60.2)
- added R9: 33, Resistor_SMD:R_0402_1005Metric, F.Cu at (415.1, 60.2)
- added R90: 33, Resistor_SMD:R_0402_1005Metric, F.Cu at (395.6, 62.2)
- added R91: 33, Resistor_SMD:R_0402_1005Metric, F.Cu at (395.6, 64.2)
- added R92: 33, Resistor_SMD:R_0402_1005Metric, F.Cu at (395.6, 66.2)
- added R93: 33, Resistor_SMD:R_0402_1005Metric, F.Cu at (395.6, 68.2)
- added R94: 33, Resistor_SMD:R_0402_1005Metric, F.Cu at (395.6, 70.2)
- added R95: 33, Resistor_SMD:R_0402_1005Metric, F.Cu at (395.6, 72.1)
- added R96: 33, Resistor_SMD:R_0402_1005Metric, F.Cu at (395.6, 74.1)
- added R97: 33, Resistor_SMD:R_0402_1005Metric, F.Cu at (395.6, 76.1)
- added R98: 33, Resistor_SMD:R_0402_1005Metric, F.Cu at (395.6, 78.1)
- added R99: 33, Resistor_SMD:R_0402_1005Metric, F.Cu at (395.6, 80.1)
- added U10: TXB0108PW, Package_SO:TSSOP-20_4.4x6.5mm_P0.65mm, F.Cu at (369.4, 79.3)
- added U100: 74LVC2G17, Package_TO_SOT_SMD:SOT-23-6, F.Cu at (227.3, 260.6)
- added U101: 74LVC2G17, Package_TO_SOT_SMD:SOT-23-6, F.Cu at (222.8, 263.2)
- added U102: 74LVC2G17, Package_TO_SOT_SMD:SOT-23-6, F.Cu at (218.4, 265.8)
- added U103: 74LVC2G17, Package_TO_SOT_SMD:SOT-23-6, F.Cu at (214.1, 268.3)
- added U104: 74LVC2G17, Package_TO_SOT_SMD:SOT-23-6, F.Cu at (209.6, 270.7)
- added U105: 74LVC2G17, Package_TO_SOT_SMD:SOT-23-6, F.Cu at (265.8, 218.3)
- added U106: 74LVC2G17, Package_TO_SOT_SMD:SOT-23-6, F.Cu at (262.0, 224.8)
- added U107: 74LVC2G17, Package_TO_SOT_SMD:SOT-23-6, F.Cu at (259.5, 229.2)
- added U108: 74LVC2G17, Package_TO_SOT_SMD:SOT-23-6, F.Cu at (257.0, 233.7)
- added U109: 74LVC2G17, Package_TO_SOT_SMD:SOT-23-6, F.Cu at (254.5, 238.0)
- added U11: TXB0108PW, Package_SO:TSSOP-20_4.4x6.5mm_P0.65mm, F.Cu at (369.4, 87.4)
- added U110: 74LVC2G17, Package_TO_SOT_SMD:SOT-23-6, F.Cu at (251.8, 242.4)
- added U12: TXB0108PW, Package_SO:TSSOP-20_4.4x6.5mm_P0.65mm, F.Cu at (369.4, 95.4)
- added U13: TXB0108PW, Package_SO:TSSOP-20_4.4x6.5mm_P0.65mm, F.Cu at (369.4, 103.5)
- added U14: TXB0108PW, Package_SO:TSSOP-20_4.4x6.5mm_P0.65mm, F.Cu at (378.2, 63.2)
- added U15: TXB0108PW, Package_SO:TSSOP-20_4.4x6.5mm_P0.65mm, F.Cu at (378.2, 71.3)
- added U16: TXB0108PW, Package_SO:TSSOP-20_4.4x6.5mm_P0.65mm, F.Cu at (378.2, 79.3)
- added U17: TXB0108PW, Package_SO:TSSOP-20_4.4x6.5mm_P0.65mm, F.Cu at (378.2, 87.4)
- added U18: TXB0108PW, Package_SO:TSSOP-20_4.4x6.5mm_P0.65mm, F.Cu at (378.2, 95.4)
- added U19: 74LVC2G17, Package_TO_SOT_SMD:SOT-23-6, F.Cu at (358.9, 109.7)
- added U20: 74LVC2G17, Package_TO_SOT_SMD:SOT-23-6, F.Cu at (358.9, 114.2)
- added U21: 74LVC2G17, Package_TO_SOT_SMD:SOT-23-6, F.Cu at (358.9, 118.6)
- added U22: 74LVC2G17, Package_TO_SOT_SMD:SOT-23-6, F.Cu at (358.9, 123.1)
- added U23: 74LVC2G17, Package_TO_SOT_SMD:SOT-23-6, F.Cu at (364.0, 109.7)
- added U24: 74LVC2G17, Package_TO_SOT_SMD:SOT-23-6, F.Cu at (364.0, 114.2)
- added U25: 74LVC2G17, Package_TO_SOT_SMD:SOT-23-6, F.Cu at (364.0, 118.6)
- added U26: 74LVC2G17, Package_TO_SOT_SMD:SOT-23-6, F.Cu at (364.0, 123.1)
- added U27: 74LVC2G17, Package_TO_SOT_SMD:SOT-23-6, F.Cu at (369.2, 109.7)
- added U28: 74LVC2G17, Package_TO_SOT_SMD:SOT-23-6, F.Cu at (369.2, 114.2)
- added U29: 74LVC2G17, Package_TO_SOT_SMD:SOT-23-6, F.Cu at (369.2, 118.6)
- added U30: 74LVC2G17, Package_TO_SOT_SMD:SOT-23-6, F.Cu at (369.2, 123.1)
- added U31: 74LVC2G17, Package_TO_SOT_SMD:SOT-23-6, F.Cu at (374.3, 109.7)
- added U32: 74LVC2G17, Package_TO_SOT_SMD:SOT-23-6, F.Cu at (374.3, 114.2)
- added U33: 74LVC2G17, Package_TO_SOT_SMD:SOT-23-6, F.Cu at (374.3, 118.6)
- added U34: 74LVC2G17, Package_TO_SOT_SMD:SOT-23-6, F.Cu at (374.3, 123.1)
- added U35: 74LVC2G17, Package_TO_SOT_SMD:SOT-23-6, F.Cu at (379.5, 109.7)
- added U36: 74LVC2G17, Package_TO_SOT_SMD:SOT-23-6, F.Cu at (379.5, 114.2)
- added U37: 74LVC2G17, Package_TO_SOT_SMD:SOT-23-6, F.Cu at (379.5, 118.6)
- added U38: 74LVC2G17, Package_TO_SOT_SMD:SOT-23-6, F.Cu at (379.5, 123.1)
- added U39: 74LVC2G17, Package_TO_SOT_SMD:SOT-23-6, F.Cu at (274.3, 168.9)
- added U40: 74LVC2G17, Package_TO_SOT_SMD:SOT-23-6, F.Cu at (274.2, 176.4)
- added U41: 74LVC2G17, Package_TO_SOT_SMD:SOT-23-6, F.Cu at (274.2, 181.5)
- added U42: 74LVC2G17, Package_TO_SOT_SMD:SOT-23-6, F.Cu at (274.3, 186.6)
- added U43: 74LVC2G17, Package_TO_SOT_SMD:SOT-23-6, F.Cu at (274.3, 191.6)
- added U44: 74LVC2G17, Package_TO_SOT_SMD:SOT-23-6, F.Cu at (274.2, 196.7)
- added U45: 74LVC2G17, Package_TO_SOT_SMD:SOT-23-6, F.Cu at (256.9, 121.8)
- added U46: 74LVC2G17, Package_TO_SOT_SMD:SOT-23-6, F.Cu at (260.6, 128.3)
- added U47: 74LVC2G17, Package_TO_SOT_SMD:SOT-23-6, F.Cu at (263.2, 132.8)
- added U48: 74LVC2G17, Package_TO_SOT_SMD:SOT-23-6, F.Cu at (265.8, 137.2)
- added U49: 74LVC2G17, Package_TO_SOT_SMD:SOT-23-6, F.Cu at (268.3, 141.5)
- added U50: 74LVC2G17, Package_TO_SOT_SMD:SOT-23-6, F.Cu at (270.7, 146.0)
- added U51: 74LVC2G17, Package_TO_SOT_SMD:SOT-23-6, F.Cu at (218.3, 89.8)
- added U52: 74LVC2G17, Package_TO_SOT_SMD:SOT-23-6, F.Cu at (224.8, 93.6)
- added U53: 74LVC2G17, Package_TO_SOT_SMD:SOT-23-6, F.Cu at (229.2, 96.1)
- added U54: 74LVC2G17, Package_TO_SOT_SMD:SOT-23-6, F.Cu at (233.7, 98.6)
- added U55: 74LVC2G17, Package_TO_SOT_SMD:SOT-23-6, F.Cu at (238.0, 101.1)
- added U56: 74LVC2G17, Package_TO_SOT_SMD:SOT-23-6, F.Cu at (242.4, 103.8)
- added U57: 74LVC2G17, Package_TO_SOT_SMD:SOT-23-6, F.Cu at (168.9, 81.3)
- added U58: 74LVC2G17, Package_TO_SOT_SMD:SOT-23-6, F.Cu at (176.4, 81.4)
- added U59: 74LVC2G17, Package_TO_SOT_SMD:SOT-23-6, F.Cu at (181.5, 81.4)
- added U60: 74LVC2G17, Package_TO_SOT_SMD:SOT-23-6, F.Cu at (186.6, 81.3)
- added U61: 74LVC2G17, Package_TO_SOT_SMD:SOT-23-6, F.Cu at (191.6, 81.3)
- added U62: 74LVC2G17, Package_TO_SOT_SMD:SOT-23-6, F.Cu at (196.7, 81.4)
- added U63: 74LVC2G17, Package_TO_SOT_SMD:SOT-23-6, F.Cu at (121.8, 98.7)
- added U64: 74LVC2G17, Package_TO_SOT_SMD:SOT-23-6, F.Cu at (128.3, 95.0)
- added U65: 74LVC2G17, Package_TO_SOT_SMD:SOT-23-6, F.Cu at (132.8, 92.4)
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- renumbered C11 to C1, C20 to C10, C21 to C11, C22 to C12, C12 to C2, C13 to C3, C14 to C4, C15 to C5, C16 to C6, C17 to C7, C18 to C8, C19 to C9, Q2 to Q1
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Connections:
- net Net-(SW1-A) renamed /Power & Voltage Regulators/SW_5V
- C23 pad 1: +5V -> +3.3V
- J2 pad 29: /Level Shifters/PAN3V.MOSI_07 -> Net-(J2-Pin_29)
- J2 pad 30: /Level Shifters/PAN3V.MOSI_08 -> Net-(J2-Pin_30)
- J2 pad 31: /Level Shifters/PAN3V.MOSI_09 -> Net-(J2-Pin_31)
- J2 pad 32: /Level Shifters/PAN3V.MOSI_10 -> Net-(J2-Pin_32)
- J2 pad 33: /Level Shifters/PAN3V.MOSI_11 -> Net-(J2-Pin_33)
- J2 pad 34: /Level Shifters/PAN3V.RESET -> Net-(J2-Pin_34)
- J2 pad 35: /Level Shifters/PAN3V.EXT_INT -> Net-(J2-Pin_35)
- J2 pad 36: /Level Shifters/PAN3V.MISO_11 -> Net-(J2-Pin_36)
- J2 pad 37: /Level Shifters/PAN3V.MISO_10 -> Net-(J2-Pin_37)
- J2 pad 38: /Level Shifters/PAN3V.MISO_09 -> Net-(J2-Pin_38)
- J2 pad 39: /Level Shifters/PAN3V.MISO_08 -> Net-(J2-Pin_39)
- J2 pad 40: /Level Shifters/PAN3V.MISO_07 -> Net-(J2-Pin_40)
- J2 pad 41: /Level Shifters/PAN3V.MISO_06 -> Net-(J2-Pin_41)
- J2 pad 42: /Level Shifters/PAN3V.MOSI_06 -> Net-(J2-Pin_42)
- J2 pad 43: /Level Shifters/PAN3V.MISO_05 -> Net-(J2-Pin_43)
- J2 pad 44: /Level Shifters/PAN3V.MOSI_05 -> Net-(J2-Pin_44)
- J2 pad 45: /Level Shifters/PAN3V.MISO_04 -> Net-(J2-Pin_45)
- J2 pad 46: /Level Shifters/PAN3V.MOSI_04 -> Net-(J2-Pin_46)
- J2 pad 47: /Level Shifters/PAN3V.MISO_03 -> Net-(J2-Pin_47)
- J2 pad 48: /Level Shifters/PAN3V.MOSI_03 -> Net-(J2-Pin_48)
- J2 pad 49: /Level Shifters/PAN3V.MISO_02 -> Net-(J2-Pin_49)
- J2 pad 50: /Level Shifters/PAN3V.MOSI_02 -> /Level Shifters/PAN3V.MISO_00
- J2 pad 51: /Level Shifters/PAN3V.MISO_01 -> Net-(J2-Pin_51)
- J2 pad 52: /Level Shifters/PAN3V.MOSI_01 -> /Level Shifters/PAN3V.MISO_01
- J2 pad 53: /Level Shifters/PAN3V.MISO_00 -> Net-(J2-Pin_53)
- J2 pad 54: /Level Shifters/PAN3V.MOSI_00 -> /Level Shifters/PAN3V.MISO_02
- J2 pad 55: /Level Shifters/PAN3V.SCK_05 -> Net-(J2-Pin_55)
- J2 pad 56: /Level Shifters/PAN3V.SCK_04 -> /Level Shifters/PAN3V.MISO_03
- J2 pad 57: /Level Shifters/PAN3V.SCK_03 -> Net-(J2-Pin_57)
- J2 pad 58: /Level Shifters/PAN3V.SCK_02 -> /Level Shifters/PAN3V.MISO_04
- J2 pad 59: /Level Shifters/PAN3V.SCK_01 -> Net-(J2-Pin_59)
- J2 pad 60: /Level Shifters/PAN3V.SCK_00 -> /Level Shifters/PAN3V.MISO_05
- J2 pad 61: /Level Shifters/PAN3V.CS_07 -> Net-(J2-Pin_61)
- J2 pad 62: /Level Shifters/PAN3V.CS_06 -> /Level Shifters/PAN3V.MISO_06
- J2 pad 63: /Level Shifters/PAN3V.CS_05 -> /Level Shifters/PAN3V.MISO_07
- J2 pad 64: /Level Shifters/PAN3V.CS_04 -> /Level Shifters/PAN3V.MISO_08
- J2 pad 65: /Level Shifters/PAN3V.CS_03 -> /Level Shifters/PAN3V.MISO_09
- J2 pad 66: /Level Shifters/PAN3V.CS_02 -> /Level Shifters/PAN3V.MISO_10
- J2 pad 67: /Level Shifters/PAN3V.CS_01 -> /Level Shifters/PAN3V.MISO_11
- J2 pad 68: /Level Shifters/PAN3V.CS_00 -> Net-(J2-Pin_68)
- P1 pad 10: /Level Shifters/PAN5V.CS_03 -> /Panel Headers/CS_03_P01
- P1 pad 11: /Level Shifters/PAN5V.CS_04 -> /Panel Headers/CS_04_P01
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Routing:
- added copper zone on In2.Cu, net +5V
- added copper zone on In1.Cu, net GND
Other:
- outline, holes or cut-outs redrawn
- board text removed: "3.3V"
- board text removed: "A0"
- board text removed: "A1"
- board text removed: "ANALOG IN"
- board text removed: "GND"
- board text removed: "QWIIC/QT"
- board text removed: "SCL"
- board text removed: "SDA"
