File: development/arena_12-12/ni/ni_arena_12-12_v0p1/ni_arena_12-12.kicad_pcb (KiCad board)
At the start: 4 copper layers, 228.6 x 228.6 mm, 581 parts, among them J1 Barrel_Jack, J2 NI_TE_68pos, J3 Barrel_Jack, P1 CONN15, P10 CONN15, P11 CONN15, P12 CONN15, P2 CONN15, P3 CONN15, P4 CONN15, P5 CONN15, P6 CONN15, P7 CONN15, P8 CONN15, P9 CONN15, Q1 MOSFET_NCHAN, SW1 SW_SPDT, U1 AP2112K-3.3, U10 TXB0108PW, U100 74LVC2G17, U101 74LVC2G17, U102 74LVC2G17, U103 74LVC2G17, U104 74LVC2G17, U105 74LVC2G17, U106 74LVC2G17, U107 74LVC2G17, U108 74LVC2G17, U109 74LVC2G17, U11 TXB0108PW, U110 74LVC2G17, U12 TXB0108PW, U13 TXB0108PW, U14 TXB0108PW, U15 TXB0108PW, U16 TXB0108PW, U17 TXB0108PW, U18 TXB0108PW, U19 74LVC2G17, U2 TXB0108PW, U20 74LVC2G17, U21 74LVC2G17, U22 74LVC2G17, U23 74LVC2G17, U24 74LVC2G17, U25 74LVC2G17, U26 74LVC2G17, U27 74LVC2G17, U28 74LVC2G17, U29 74LVC2G17, U3 TXB0108PW, U30 74LVC2G17, U31 74LVC2G17, U32 74LVC2G17, U33 74LVC2G17, U34 74LVC2G17, U35 74LVC2G17, U36 74LVC2G17, U37 74LVC2G17, U38 74LVC2G17, U39 74LVC2G17, U4 TXB0108PW, U40 74LVC2G17, U41 74LVC2G17, U42 74LVC2G17, U43 74LVC2G17, U44 74LVC2G17, U45 74LVC2G17, U46 74LVC2G17, U47 74LVC2G17, U48 74LVC2G17, U49 74LVC2G17, U5 TXB0108PW, U50 74LVC2G17, U51 74LVC2G17, U52 74LVC2G17, U53 74LVC2G17, U54 74LVC2G17, U55 74LVC2G17, U56 74LVC2G17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

Commit message: Worked on layout for 12-12 ni arena with schmitt buffers.
Finished layout of components at base of panel columns.
Parts:
- removed the R163 at (476.5, -20.8)
- removed the R164 at (476.5, -18.8)
- removed the R165 at (476.5, -16.8)
- removed the R166 at (476.5, -14.8)
- removed the R167 at (476.5, -12.9)
- removed the R168 at (476.5, -10.9)
- removed the R169 at (476.5, -8.88)
- removed the R170 at (476.5, -6.89)
- removed the R171 at (476.5, -4.90)
- removed the R172 at (476.5, -2.91)
- removed the R173 at (476.5, -0.92)
- removed the R174 at (476.5, 1.07)
- added R29: 33, Resistor_SMD:R_0402_1005Metric, F.Cu at (384.0, 60.2)
- added R30: 33, Resistor_SMD:R_0402_1005Metric, F.Cu at (384.0, 62.2)
- added R31: 33, Resistor_SMD:R_0402_1005Metric, F.Cu at (384.0, 64.2)
- added R32: 33, Resistor_SMD:R_0402_1005Metric, F.Cu at (384.0, 66.2)
- added R33: 33, Resistor_SMD:R_0402_1005Metric, F.Cu at (384.0, 68.2)
- added R34: 33, Resistor_SMD:R_0402_1005Metric, F.Cu at (384.0, 70.2)
- added R35: 33, Resistor_SMD:R_0402_1005Metric, F.Cu at (384.0, 72.1)
- added R36: 33, Resistor_SMD:R_0402_1005Metric, F.Cu at (384.0, 74.1)
- added R37: 33, Resistor_SMD:R_0402_1005Metric, F.Cu at (384.0, 76.1)
- added R38: 33, Resistor_SMD:R_0402_1005Metric, F.Cu at (384.0, 78.1)
- added R39: 33, Resistor_SMD:R_0402_1005Metric, F.Cu at (384.0, 80.1)
- added R40: 33, Resistor_SMD:R_0402_1005Metric, F.Cu at (384.0, 82.1)
- moved U84 397.8 mm to (89.8, 218.4), turned to 30 degrees
- moved U85 394.5 mm to (87.3, 214.1), turned to 30 degrees
- moved U86 391.3 mm to (84.9, 209.6), turned to 30 degrees
- moved U87 384.9 mm to (137.3, 265.8), turned to 60 degrees
- moved U88 383.6 mm to (130.8, 262.0), turned to 60 degrees
- moved U75 382.1 mm to (81.3, 186.7)
- moved U89 382.0 mm to (126.4, 259.5), turned to 60 degrees
- moved U90 380.6 mm to (121.9, 257.0), turned to 60 degrees
- moved U81 379.8 mm to (98.7, 233.8), turned to 30 degrees
- moved U91 379.3 mm to (117.6, 254.5), turned to 60 degrees
- moved U92 378.1 mm to (113.2, 251.8), turned to 60 degrees
- moved C88 378.0 mm to (114.8, 249.1), turned to 60 degrees
- moved C87 377.2 mm to (119.2, 251.7), turned to 60 degrees
- moved C86 376.4 mm to (123.6, 254.2), turned to 60 degrees
- moved U82 376.2 mm to (95.0, 227.3), turned to 30 degrees
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- renumbered R29 to R163, R30 to R164, R31 to R165, R32 to R166, R33 to R167, R34 to R168, R35 to R169, R36 to R170, R37 to R171, R38 to R172, R39 to R173, R40 to R174
Connections:
- R100 pad 1: /Level Shifters/PAN5V.CS_4_P12 -> /Level Shifters/PAN5V.CS_5_P12
- R100 pad 2: Net-(U9-B4) -> Net-(U10-B8)
- R101 pad 1: /Level Shifters/PAN5V.CS_5_P01 -> /Level Shifters/PAN5V.CS_6_P01
- R101 pad 2: Net-(U9-B5) -> Net-(U11-B1)
- R102 pad 1: /Level Shifters/PAN5V.CS_5_P02 -> /Level Shifters/PAN5V.CS_6_P02
- R102 pad 2: Net-(U9-B6) -> Net-(U11-B2)
- R103 pad 1: /Level Shifters/PAN5V.CS_5_P03 -> /Level Shifters/PAN5V.CS_6_P03
- R103 pad 2: Net-(U9-B7) -> Net-(U11-B3)
- R104 pad 1: /Level Shifters/PAN5V.CS_5_P04 -> /Level Shifters/PAN5V.CS_6_P04
- R104 pad 2: Net-(U9-B8) -> Net-(U11-B4)
- R105 pad 1: /Level Shifters/PAN5V.CS_5_P05 -> /Level Shifters/PAN5V.CS_6_P05
- R105 pad 2: Net-(U10-B1) -> Net-(U11-B5)
- R106 pad 1: /Level Shifters/PAN5V.CS_5_P06 -> /Level Shifters/PAN5V.CS_6_P06
- R106 pad 2: Net-(U10-B2) -> Net-(U11-B6)
- R107 pad 1: /Level Shifters/PAN5V.CS_5_P07 -> /Level Shifters/PAN5V.CS_6_P07
- R107 pad 2: Net-(U10-B3) -> Net-(U11-B7)
- R108 pad 1: /Level Shifters/PAN5V.CS_5_P08 -> /Level Shifters/PAN5V.CS_6_P08
- R108 pad 2: Net-(U10-B4) -> Net-(U11-B8)
- R109 pad 1: /Level Shifters/PAN5V.CS_5_P09 -> /Level Shifters/PAN5V.CS_6_P09
- R109 pad 2: Net-(U10-B5) -> Net-(U12-B1)
- R110 pad 1: /Level Shifters/PAN5V.CS_5_P10 -> /Level Shifters/PAN5V.CS_6_P10
- R110 pad 2: Net-(U10-B6) -> Net-(U12-B2)
- R111 pad 1: /Level Shifters/PAN5V.CS_5_P11 -> /Level Shifters/PAN5V.CS_6_P11
- R111 pad 2: Net-(U10-B7) -> Net-(U12-B3)
- R112 pad 1: /Level Shifters/PAN5V.CS_5_P12 -> /Level Shifters/PAN5V.CS_6_P12
- R112 pad 2: Net-(U10-B8) -> Net-(U12-B4)
- R113 pad 1: /Level Shifters/PAN5V.CS_6_P01 -> /Level Shifters/PAN5V.CS_7_P01
- R113 pad 2: Net-(U11-B1) -> Net-(U12-B5)
- R114 pad 1: /Level Shifters/PAN5V.CS_6_P02 -> /Level Shifters/PAN5V.CS_7_P02
- R114 pad 2: Net-(U11-B2) -> Net-(U12-B6)
- R115 pad 1: /Level Shifters/PAN5V.CS_6_P03 -> /Level Shifters/PAN5V.CS_7_P03
- R115 pad 2: Net-(U11-B3) -> Net-(U12-B7)
- R116 pad 1: /Level Shifters/PAN5V.CS_6_P04 -> /Level Shifters/PAN5V.CS_7_P04
- R116 pad 2: Net-(U11-B4) -> Net-(U12-B8)
- R117 pad 1: /Level Shifters/PAN5V.CS_6_P05 -> /Level Shifters/PAN5V.CS_7_P05
- R117 pad 2: Net-(U11-B5) -> Net-(U13-B1)
- R118 pad 1: /Level Shifters/PAN5V.CS_6_P06 -> /Level Shifters/PAN5V.CS_7_P06
- R118 pad 2: Net-(U11-B6) -> Net-(U13-B2)
- R119 pad 1: /Level Shifters/PAN5V.CS_6_P07 -> /Level Shifters/PAN5V.CS_7_P07
- R119 pad 2: Net-(U11-B7) -> Net-(U13-B3)
- R120 pad 1: /Level Shifters/PAN5V.CS_6_P08 -> /Level Shifters/PAN5V.CS_7_P08
- R120 pad 2: Net-(U11-B8) -> Net-(U13-B4)
- R121 pad 1: /Level Shifters/PAN5V.CS_6_P09 -> /Level Shifters/PAN5V.CS_7_P09
- R121 pad 2: Net-(U12-B1) -> Net-(U13-B5)
- R122 pad 1: /Level Shifters/PAN5V.CS_6_P10 -> /Level Shifters/PAN5V.CS_7_P10
- R122 pad 2: Net-(U12-B2) -> Net-(U13-B6)
- R123 pad 1: /Level Shifters/PAN5V.CS_6_P11 -> /Level Shifters/PAN5V.CS_7_P11
- R123 pad 2: Net-(U12-B3) -> Net-(U13-B7)
- R124 pad 1: /Level Shifters/PAN5V.CS_6_P12 -> /Level Shifters/PAN5V.CS_7_P12
- R124 pad 2: Net-(U12-B4) -> Net-(U13-B8)
- R125 pad 1: /Level Shifters/PAN5V.CS_7_P01 -> /Level Shifters/PAN5V.SCK_0_H1
- R125 pad 2: Net-(U12-B5) -> Net-(U14-B1)
- R126 pad 1: /Level Shifters/PAN5V.CS_7_P02 -> /Level Shifters/PAN5V.SCK_0_H2
- R126 pad 2: Net-(U12-B6) -> Net-(U14-B2)
- R127 pad 1: /Level Shifters/PAN5V.CS_7_P03 -> /Level Shifters/PAN5V.SCK_1_H1
- R127 pad 2: Net-(U12-B7) -> Net-(U14-B3)
- R128 pad 1: /Level Shifters/PAN5V.CS_7_P04 -> /Level Shifters/PAN5V.SCK_1_H2
- R128 pad 2: Net-(U12-B8) -> Net-(U14-B4)
- R129 pad 1: /Level Shifters/PAN5V.CS_7_P05 -> /Level Shifters/PAN5V.SCK_2_H1
- R129 pad 2: Net-(U13-B1) -> Net-(U14-B5)
- R130 pad 1: /Level Shifters/PAN5V.CS_7_P06 -> /Level Shifters/PAN5V.SCK_2_H2
- R130 pad 2: Net-(U13-B2) -> Net-(U14-B6)
- R131 pad 1: /Level Shifters/PAN5V.CS_7_P07 -> /Level Shifters/PAN5V.SCK_3_H1
- R131 pad 2: Net-(U13-B3) -> Net-(U14-B7)
- R132 pad 1: /Level Shifters/PAN5V.CS_7_P08 -> /Level Shifters/PAN5V.SCK_3_H2
- R132 pad 2: Net-(U13-B4) -> Net-(U14-B8)
- R133 pad 1: /Level Shifters/PAN5V.CS_7_P09 -> /Level Shifters/PAN5V.SCK_4_H1
- R133 pad 2: Net-(U13-B5) -> Net-(U15-B1)
- R134 pad 1: /Level Shifters/PAN5V.CS_7_P10 -> /Level Shifters/PAN5V.SCK_4_H2
- R134 pad 2: Net-(U13-B6) -> Net-(U15-B2)
- R135 pad 1: /Level Shifters/PAN5V.CS_7_P11 -> /Level Shifters/PAN5V.SCK_5_H1
- R135 pad 2: Net-(U13-B7) -> Net-(U15-B3)
- R136 pad 1: /Level Shifters/PAN5V.CS_7_P12 -> /Level Shifters/PAN5V.SCK_5_H2
- R136 pad 2: Net-(U13-B8) -> Net-(U15-B4)
- R137 pad 1: /Level Shifters/PAN5V.SCK_0_H1 -> /Level Shifters/PAN5V.MOSI_00
- R137 pad 2: Net-(U14-B1) -> Net-(U15-B5)
- R138 pad 1: /Level Shifters/PAN5V.SCK_0_H2 -> /Level Shifters/PAN5V.MOSI_01
- R138 pad 2: Net-(U14-B2) -> Net-(U15-B6)
- R139 pad 1: /Level Shifters/PAN5V.SCK_1_H1 -> /Level Shifters/PAN5V.MOSI_02
- R139 pad 2: Net-(U14-B3) -> Net-(U15-B7)
- R140 pad 1: /Level Shifters/PAN5V.SCK_1_H2 -> /Level Shifters/PAN5V.MOSI_03
- R140 pad 2: Net-(U14-B4) -> Net-(U15-B8)
- R141 pad 1: /Level Shifters/PAN5V.SCK_2_H1 -> /Level Shifters/PAN5V.MOSI_04
- R141 pad 2: Net-(U14-B5) -> Net-(U16-B1)
- R142 pad 1: /Level Shifters/PAN5V.SCK_2_H2 -> /Level Shifters/PAN5V.MOSI_05
- R142 pad 2: Net-(U14-B6) -> Net-(U16-B2)
- R143 pad 1: /Level Shifters/PAN5V.SCK_3_H1 -> /Level Shifters/PAN5V.MOSI_06
- R143 pad 2: Net-(U14-B7) -> Net-(U16-B3)
- R144 pad 1: /Level Shifters/PAN5V.SCK_3_H2 -> /Level Shifters/PAN5V.MOSI_07
- R144 pad 2: Net-(U14-B8) -> Net-(U16-B4)
- R145 pad 1: /Level Shifters/PAN5V.SCK_4_H1 -> /Level Shifters/PAN5V.MOSI_08
- R145 pad 2: Net-(U15-B1) -> Net-(U16-B5)
- R146 pad 1: /Level Shifters/PAN5V.SCK_4_H2 -> /Level Shifters/PAN5V.MOSI_09
- R146 pad 2: Net-(U15-B2) -> Net-(U16-B6)
- R147 pad 1: /Level Shifters/PAN5V.SCK_5_H1 -> /Level Shifters/PAN5V.MOSI_10
- R147 pad 2: Net-(U15-B3) -> Net-(U16-B7)
- R148 pad 1: /Level Shifters/PAN5V.SCK_5_H2 -> /Level Shifters/PAN5V.MOSI_11
- R148 pad 2: Net-(U15-B4) -> Net-(U16-B8)
- R149 pad 1: /Level Shifters/PAN5V.MOSI_00 -> Net-(U17-A1)
- R149 pad 2: Net-(U15-B5) -> /Level Shifters/PAN3V.MISO_00
- R150 pad 1: /Level Shifters/PAN5V.MOSI_01 -> Net-(U17-A2)
- R150 pad 2: Net-(U15-B6) -> /Level Shifters/PAN3V.MISO_01
- R151 pad 1: /Level Shifters/PAN5V.MOSI_02 -> Net-(U17-A3)
- R151 pad 2: Net-(U15-B7) -> /Level Shifters/PAN3V.MISO_02
- R152 pad 1: /Level Shifters/PAN5V.MOSI_03 -> Net-(U17-A4)
- R152 pad 2: Net-(U15-B8) -> /Level Shifters/PAN3V.MISO_03
- R153 pad 1: /Level Shifters/PAN5V.MOSI_04 -> Net-(U17-A5)
- R153 pad 2: Net-(U16-B1) -> /Level Shifters/PAN3V.MISO_04
- R154 pad 1: /Level Shifters/PAN5V.MOSI_05 -> Net-(U17-A6)
- R154 pad 2: Net-(U16-B2) -> /Level Shifters/PAN3V.MISO_05
- R155 pad 1: /Level Shifters/PAN5V.MOSI_06 -> Net-(U17-A7)
- R155 pad 2: Net-(U16-B3) -> /Level Shifters/PAN3V.MISO_06
- R156 pad 1: /Level Shifters/PAN5V.MOSI_07 -> Net-(U17-A8)
- R156 pad 2: Net-(U16-B4) -> /Level Shifters/PAN3V.MISO_07
- R157 pad 1: /Level Shifters/PAN5V.MOSI_08 -> /Level Shifters/PAN5V.EXT_INT
- R157 pad 2: Net-(U16-B5) -> Net-(U18-B5)
- R158 pad 1: /Level Shifters/PAN5V.MOSI_09 -> /Level Shifters/PAN5V.RESET
- R158 pad 2: Net-(U16-B6) -> Net-(U18-B6)
- R159 pad 1: /Level Shifters/PAN5V.MOSI_10 -> /Level Shifters/PAN3V.MISO_08
- R159 pad 2: Net-(U16-B7) -> Net-(U18-A1)
- R160 pad 1: /Level Shifters/PAN5V.MOSI_11 -> /Level Shifters/PAN3V.MISO_09
- R160 pad 2: Net-(U16-B8) -> Net-(U18-A2)
- R161 pad 1: Net-(U17-A1) -> /Level Shifters/PAN3V.MISO_10
- R161 pad 2: /Level Shifters/PAN3V.MISO_00 -> Net-(U18-A3)
- R162 pad 1: Net-(U17-A2) -> /Level Shifters/PAN3V.MISO_11
- R162 pad 2: /Level Shifters/PAN3V.MISO_01 -> Net-(U18-A4)
- R41 pad 1: /Level Shifters/PAN5V.CS_0_P01 -> /Level Shifters/PAN5V.CS_1_P01
- R41 pad 2: Net-(U2-B1) -> Net-(U3-B5)
- R42 pad 1: /Level Shifters/PAN5V.CS_0_P02 -> /Level Shifters/PAN5V.CS_1_P02
- R42 pad 2: Net-(U2-B2) -> Net-(U3-B6)
- R43 pad 1: /Level Shifters/PAN5V.CS_0_P03 -> /Level Shifters/PAN5V.CS_1_P03
- R43 pad 2: Net-(U2-B3) -> Net-(U3-B7)
- R44 pad 1: /Level Shifters/PAN5V.CS_0_P04 -> /Level Shifters/PAN5V.CS_1_P04
- R44 pad 2: Net-(U2-B4) -> Net-(U3-B8)
- R45 pad 1: /Level Shifters/PAN5V.CS_0_P05 -> /Level Shifters/PAN5V.CS_1_P05
- R45 pad 2: Net-(U2-B5) -> Net-(U4-B1)
- R46 pad 1: /Level Shifters/PAN5V.CS_0_P06 -> /Level Shifters/PAN5V.CS_1_P06
- R46 pad 2: Net-(U2-B6) -> Net-(U4-B2)
- R47 pad 1: /Level Shifters/PAN5V.CS_0_P07 -> /Level Shifters/PAN5V.CS_1_P07
- R47 pad 2: Net-(U2-B7) -> Net-(U4-B3)
- R48 pad 1: /Level Shifters/PAN5V.CS_0_P08 -> /Level Shifters/PAN5V.CS_1_P08
- R48 pad 2: Net-(U2-B8) -> Net-(U4-B4)
- R49 pad 1: /Level Shifters/PAN5V.CS_0_P09 -> /Level Shifters/PAN5V.CS_1_P09
- R49 pad 2: Net-(U3-B1) -> Net-(U4-B5)
- R50 pad 1: /Level Shifters/PAN5V.CS_0_P10 -> /Level Shifters/PAN5V.CS_1_P10
- R50 pad 2: Net-(U3-B2) -> Net-(U4-B6)
- R51 pad 1: /Level Shifters/PAN5V.CS_0_P11 -> /Level Shifters/PAN5V.CS_1_P11
- R51 pad 2: Net-(U3-B3) -> Net-(U4-B7)
- R52 pad 1: /Level Shifters/PAN5V.CS_0_P12 -> /Level Shifters/PAN5V.CS_1_P12
- R52 pad 2: Net-(U3-B4) -> Net-(U4-B8)
- R53 pad 1: /Level Shifters/PAN5V.CS_1_P01 -> /Level Shifters/PAN5V.CS_2_P01
- R53 pad 2: Net-(U3-B5) -> Net-(U5-B1)
- R54 pad 1: /Level Shifters/PAN5V.CS_1_P02 -> /Level Shifters/PAN5V.CS_2_P02
- R54 pad 2: Net-(U3-B6) -> Net-(U5-B2)
- R55 pad 1: /Level Shifters/PAN5V.CS_1_P03 -> /Level Shifters/PAN5V.CS_2_P03
- R55 pad 2: Net-(U3-B7) -> Net-(U5-B3)
- R56 pad 1: /Level Shifters/PAN5V.CS_1_P04 -> /Level Shifters/PAN5V.CS_2_P04
- R56 pad 2: Net-(U3-B8) -> Net-(U5-B4)
- R57 pad 1: /Level Shifters/PAN5V.CS_1_P05 -> /Level Shifters/PAN5V.CS_2_P05
- R57 pad 2: Net-(U4-B1) -> Net-(U5-B5)
- R58 pad 1: /Level Shifters/PAN5V.CS_1_P06 -> /Level Shifters/PAN5V.CS_2_P06
- R58 pad 2: Net-(U4-B2) -> Net-(U5-B6)
- R59 pad 1: /Level Shifters/PAN5V.CS_1_P07 -> /Level Shifters/PAN5V.CS_2_P07
- R59 pad 2: Net-(U4-B3) -> Net-(U5-B7)
- R60 pad 1: /Level Shifters/PAN5V.CS_1_P08 -> /Level Shifters/PAN5V.CS_2_P08
- R60 pad 2: Net-(U4-B4) -> Net-(U5-B8)
- R61 pad 1: /Level Shifters/PAN5V.CS_1_P09 -> /Level Shifters/PAN5V.CS_2_P09
- R61 pad 2: Net-(U4-B5) -> Net-(U6-B1)
- R62 pad 1: /Level Shifters/PAN5V.CS_1_P10 -> /Level Shifters/PAN5V.CS_2_P10
- R62 pad 2: Net-(U4-B6) -> Net-(U6-B2)
- R63 pad 1: /Level Shifters/PAN5V.CS_1_P11 -> /Level Shifters/PAN5V.CS_2_P11
- R63 pad 2: Net-(U4-B7) -> Net-(U6-B3)
- R64 pad 1: /Level Shifters/PAN5V.CS_1_P12 -> /Level Shifters/PAN5V.CS_2_P12
- R64 pad 2: Net-(U4-B8) -> Net-(U6-B4)
- R65 pad 1: /Level Shifters/PAN5V.CS_2_P01 -> /Level Shifters/PAN5V.CS_3_P01
- R65 pad 2: Net-(U5-B1) -> Net-(U6-B5)
- R66 pad 1: /Level Shifters/PAN5V.CS_2_P02 -> /Level Shifters/PAN5V.CS_3_P02
- R66 pad 2: Net-(U5-B2) -> Net-(U6-B6)
- R67 pad 1: /Level Shifters/PAN5V.CS_2_P03 -> /Level Shifters/PAN5V.CS_3_P03
- R67 pad 2: Net-(U5-B3) -> Net-(U6-B7)
- R68 pad 1: /Level Shifters/PAN5V.CS_2_P04 -> /Level Shifters/PAN5V.CS_3_P04
- R68 pad 2: Net-(U5-B4) -> Net-(U6-B8)
- R69 pad 1: /Level Shifters/PAN5V.CS_2_P05 -> /Level Shifters/PAN5V.CS_3_P05
- R69 pad 2: Net-(U5-B5) -> Net-(U7-B1)
- R70 pad 1: /Level Shifters/PAN5V.CS_2_P06 -> /Level Shifters/PAN5V.CS_3_P06
- R70 pad 2: Net-(U5-B6) -> Net-(U7-B2)
- R71 pad 1: /Level Shifters/PAN5V.CS_2_P07 -> /Level Shifters/PAN5V.CS_3_P07
- R71 pad 2: Net-(U5-B7) -> Net-(U7-B3)
- R72 pad 1: /Level Shifters/PAN5V.CS_2_P08 -> /Level Shifters/PAN5V.CS_3_P08
- R72 pad 2: Net-(U5-B8) -> Net-(U7-B4)
- R73 pad 1: /Level Shifters/PAN5V.CS_2_P09 -> /Level Shifters/PAN5V.CS_3_P09
- R73 pad 2: Net-(U6-B1) -> Net-(U7-B5)
- R74 pad 1: /Level Shifters/PAN5V.CS_2_P10 -> /Level Shifters/PAN5V.CS_3_P10
- R74 pad 2: Net-(U6-B2) -> Net-(U7-B6)
- R75 pad 1: /Level Shifters/PAN5V.CS_2_P11 -> /Level Shifters/PAN5V.CS_3_P11
- R75 pad 2: Net-(U6-B3) -> Net-(U7-B7)
- R76 pad 1: /Level Shifters/PAN5V.CS_2_P12 -> /Level Shifters/PAN5V.CS_3_P12
- R76 pad 2: Net-(U6-B4) -> Net-(U7-B8)
- R77 pad 1: /Level Shifters/PAN5V.CS_3_P01 -> /Level Shifters/PAN5V.CS_4_P01
- R77 pad 2: Net-(U6-B5) -> Net-(U8-B1)
- R78 pad 1: /Level Shifters/PAN5V.CS_3_P02 -> /Level Shifters/PAN5V.CS_4_P02
- R78 pad 2: Net-(U6-B6) -> Net-(U8-B2)
- R79 pad 1: /Level Shifters/PAN5V.CS_3_P03 -> /Level Shifters/PAN5V.CS_4_P03
- R79 pad 2: Net-(U6-B7) -> Net-(U8-B3)
- R80 pad 1: /Level Shifters/PAN5V.CS_3_P04 -> /Level Shifters/PAN5V.CS_4_P04
- R80 pad 2: Net-(U6-B8) -> Net-(U8-B4)
- R81 pad 1: /Level Shifters/PAN5V.CS_3_P05 -> /Level Shifters/PAN5V.CS_4_P05
- R81 pad 2: Net-(U7-B1) -> Net-(U8-B5)
- R82 pad 1: /Level Shifters/PAN5V.CS_3_P06 -> /Level Shifters/PAN5V.CS_4_P06
- R82 pad 2: Net-(U7-B2) -> Net-(U8-B6)
- R83 pad 1: /Level Shifters/PAN5V.CS_3_P07 -> /Level Shifters/PAN5V.CS_4_P07
- R83 pad 2: Net-(U7-B3) -> Net-(U8-B7)
- R84 pad 1: /Level Shifters/PAN5V.CS_3_P08 -> /Level Shifters/PAN5V.CS_4_P08
- R84 pad 2: Net-(U7-B4) -> Net-(U8-B8)
- R85 pad 1: /Level Shifters/PAN5V.CS_3_P09 -> /Level Shifters/PAN5V.CS_4_P09
- R85 pad 2: Net-(U7-B5) -> Net-(U9-B1)
- R86 pad 1: /Level Shifters/PAN5V.CS_3_P10 -> /Level Shifters/PAN5V.CS_4_P10
- R86 pad 2: Net-(U7-B6) -> Net-(U9-B2)
- R87 pad 1: /Level Shifters/PAN5V.CS_3_P11 -> /Level Shifters/PAN5V.CS_4_P11
- R87 pad 2: Net-(U7-B7) -> Net-(U9-B3)
- R88 pad 1: /Level Shifters/PAN5V.CS_3_P12 -> /Level Shifters/PAN5V.CS_4_P12
- R88 pad 2: Net-(U7-B8) -> Net-(U9-B4)
- R89 pad 1: /Level Shifters/PAN5V.CS_4_P01 -> /Level Shifters/PAN5V.CS_5_P01
- R89 pad 2: Net-(U8-B1) -> Net-(U9-B5)
- R90 pad 1: /Level Shifters/PAN5V.CS_4_P02 -> /Level Shifters/PAN5V.CS_5_P02
- R90 pad 2: Net-(U8-B2) -> Net-(U9-B6)
- R91 pad 1: /Level Shifters/PAN5V.CS_4_P03 -> /Level Shifters/PAN5V.CS_5_P03
- R91 pad 2: Net-(U8-B3) -> Net-(U9-B7)
- R92 pad 1: /Level Shifters/PAN5V.CS_4_P04 -> /Level Shifters/PAN5V.CS_5_P04
- R92 pad 2: Net-(U8-B4) -> Net-(U9-B8)
- R93 pad 1: /Level Shifters/PAN5V.CS_4_P05 -> /Level Shifters/PAN5V.CS_5_P05
- R93 pad 2: Net-(U8-B5) -> Net-(U10-B1)
- R94 pad 1: /Level Shifters/PAN5V.CS_4_P06 -> /Level Shifters/PAN5V.CS_5_P06
- R94 pad 2: Net-(U8-B6) -> Net-(U10-B2)
- R95 pad 1: /Level Shifters/PAN5V.CS_4_P07 -> /Level Shifters/PAN5V.CS_5_P07
- R95 pad 2: Net-(U8-B7) -> Net-(U10-B3)
- R96 pad 1: /Level Shifters/PAN5V.CS_4_P08 -> /Level Shifters/PAN5V.CS_5_P08
- R96 pad 2: Net-(U8-B8) -> Net-(U10-B4)
- R97 pad 1: /Level Shifters/PAN5V.CS_4_P09 -> /Level Shifters/PAN5V.CS_5_P09
- R97 pad 2: Net-(U9-B1) -> Net-(U10-B5)
- R98 pad 1: /Level Shifters/PAN5V.CS_4_P10 -> /Level Shifters/PAN5V.CS_5_P10
- R98 pad 2: Net-(U9-B2) -> Net-(U10-B6)
- R99 pad 1: /Level Shifters/PAN5V.CS_4_P11 -> /Level Shifters/PAN5V.CS_5_P11
- R99 pad 2: Net-(U9-B3) -> Net-(U10-B7)

Commit message: Worked on layout for 12-12 NI arena /w schmitt buffers.
Parts:
- moved C114 361.1 mm to (193.1, 406.7)
- moved C116 361.1 mm to (193.1, 410.7)
- moved C16 361.1 mm to (187.4, 394.9)
- moved R56 361.1 mm to (190.3, 387.0)
- moved R57 361.1 mm to (190.3, 389.0)
- moved R59 361.1 mm to (193.2, 363.1)
- moved R65 361.1 mm to (193.2, 375.0)
- moved R71 361.1 mm to (193.2, 387.0)
- moved R72 361.1 mm to (193.2, 389.0)
- moved R74 361.1 mm to (196.1, 363.1)
- moved C113 361.1 mm to (193.1, 404.8)
- moved C115 361.1 mm to (193.1, 408.7)
- moved C117 361.1 mm to (196.0, 392.9)
- moved C118 361.1 mm to (196.0, 394.9)
- moved R53 361.1 mm to (190.3, 381.0)
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Connections:
- C28 pad 1: +3.3V -> +5V
- C29 pad 1: +3.3V -> +5V
- C30 pad 1: +3.3V -> +5V
- C31 pad 1: +3.3V -> +5V
- C32 pad 1: +3.3V -> +5V
- C33 pad 1: +3.3V -> +5V
- U28 pad 5: +3.3V -> +5V
- U29 pad 5: +3.3V -> +5V
- U30 pad 5: +3.3V -> +5V
- U31 pad 5: +3.3V -> +5V
- U36 pad 1: /Level Shifters/PAN5V.MISO_08 -> /Level Shifters/PAN5V.MISO_09
- U36 pad 3: /Level Shifters/PAN5V.MISO_09 -> /Level Shifters/PAN5V.MISO_08
- U36 pad 4: Net-(U18-B2) -> Net-(U18-B1)
- U36 pad 5: +3.3V -> +5V
- U36 pad 6: Net-(U18-B1) -> Net-(U18-B2)
- U37 pad 1: /Level Shifters/PAN5V.MISO_10 -> /Level Shifters/PAN5V.MISO_11
- U37 pad 3: /Level Shifters/PAN5V.MISO_11 -> /Level Shifters/PAN5V.MISO_10
- U37 pad 4: Net-(U18-B4) -> Net-(U18-B3)
- U37 pad 5: +3.3V -> +5V
- U37 pad 6: Net-(U18-B3) -> Net-(U18-B4)
