File: development/arena_12-12/ni/ni_arena_12-12_v0p1/panel_headers.kicad_sch (KiCad schematic)
At the start: 315 parts, among them P1 CONN15, P10 CONN15, P11 CONN15, P12 CONN15, P2 CONN15, P3 CONN15, P4 CONN15, P5 CONN15, P6 CONN15, P7 CONN15, P8 CONN15, P9 CONN15, Q1 MOSFET_NCHAN, U100 74LVC2G17, U101 74LVC2G17, U102 74LVC2G17, U103 74LVC2G17, U104 74LVC2G17, U105 74LVC2G17, U106 74LVC2G17, U107 74LVC2G17, U108 74LVC2G17, U109 74LVC2G17, U110 74LVC2G17, U39 74LVC2G17, U40 74LVC2G17, U41 74LVC2G17, U42 74LVC2G17, U43 74LVC2G17, U44 74LVC2G17, U45 74LVC2G17, U46 74LVC2G17, U47 74LVC2G17, U48 74LVC2G17, U49 74LVC2G17, U50 74LVC2G17, U51 74LVC2G17, U52 74LVC2G17, U53 74LVC2G17, U54 74LVC2G17, U55 74LVC2G17, U56 74LVC2G17, U57 74LVC2G17, U58 74LVC2G17, U59 74LVC2G17, U60 74LVC2G17, U61 74LVC2G17, U62 74LVC2G17, U63 74LVC2G17, U64 74LVC2G17, U65 74LVC2G17, U66 74LVC2G17, U67 74LVC2G17, U68 74LVC2G17, U69 74LVC2G17, U70 74LVC2G17, U71 74LVC2G17, U72 74LVC2G17, U73 74LVC2G17, U74 74LVC2G17, U75 74LVC2G17, U76 74LVC2G17, U77 74LVC2G17, U78 74LVC2G17, U79 74LVC2G17, U80 74LVC2G17, U81 74LVC2G17, U82 74LVC2G17, U83 74LVC2G17, U84 74LVC2G17, U85 74LVC2G17, U86 74LVC2G17, U87 74LVC2G17, U88 74LVC2G17, U89 74LVC2G17, U90 74LVC2G17, U91 74LVC2G17, U92 74LVC2G17, U93 74LVC2G17, U94 74LVC2G17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

Commit message: Finished preliminary hand routing for NI 12-12 arena.
Connections:
- net PAN5V.CS_0_P02: now also U46.3; no longer U46.1
- net PAN5V.CS_0_P03: now also U52.3; no longer U52.1
- net PAN5V.CS_0_P04: now also U58.3; no longer U58.1
- net PAN5V.CS_0_P05: now also U64.3; no longer U64.1
- net PAN5V.CS_0_P06: now also U70.3; no longer U70.1
- net PAN5V.CS_0_P07: now also U76.3; no longer U76.1
- net PAN5V.CS_0_P08: now also U82.3; no longer U82.1
- net PAN5V.CS_0_P09: now also U88.3; no longer U88.1
- net PAN5V.CS_0_P10: now also U94.3; no longer U94.1
- net PAN5V.CS_0_P11: now also U100.3; no longer U100.1
- net PAN5V.CS_0_P12: now also U106.3; no longer U106.1
- net PAN5V.CS_1_P02: now also U46.1; no longer U46.3
- net PAN5V.CS_1_P03: now also U52.1; no longer U52.3
- net PAN5V.CS_1_P04: now also U58.1; no longer U58.3
- net PAN5V.CS_1_P05: now also U64.1; no longer U64.3
- net PAN5V.CS_1_P06: now also U70.1; no longer U70.3
- net PAN5V.CS_1_P07: now also U76.1; no longer U76.3
- net PAN5V.CS_1_P08: now also U82.1; no longer U82.3
- net PAN5V.CS_1_P09: now also U88.1; no longer U88.3
- net PAN5V.CS_1_P10: now also U94.1; no longer U94.3
- net PAN5V.CS_1_P11: now also U100.1; no longer U100.3
- net PAN5V.CS_1_P12: now also U106.1; no longer U106.3
- net PAN5V.CS_2_P02: now also U47.3; no longer U47.1
- net PAN5V.CS_2_P03: now also U53.3; no longer U53.1
- net PAN5V.CS_2_P04: now also U59.3; no longer U59.1
- net PAN5V.CS_2_P05: now also U65.3; no longer U65.1
- net PAN5V.CS_2_P06: now also U71.3; no longer U71.1
- net PAN5V.CS_2_P07: now also U77.3; no longer U77.1
- net PAN5V.CS_2_P08: now also U83.3; no longer U83.1
- net PAN5V.CS_2_P09: now also U89.3; no longer U89.1
- net PAN5V.CS_2_P10: now also U95.3; no longer U95.1
- net PAN5V.CS_2_P11: now also U101.3; no longer U101.1
- net PAN5V.CS_2_P12: now also U107.3; no longer U107.1
- net PAN5V.CS_3_P02: now also U47.1; no longer U47.3
- net PAN5V.CS_3_P03: now also U53.1; no longer U53.3
- net PAN5V.CS_3_P04: now also U59.1; no longer U59.3
- net PAN5V.CS_3_P05: now also U65.1; no longer U65.3
- net PAN5V.CS_3_P06: now also U71.1; no longer U71.3
- net PAN5V.CS_3_P07: now also U77.1; no longer U77.3
- net PAN5V.CS_3_P08: now also U83.1; no longer U83.3
- net PAN5V.CS_3_P09: now also U89.1; no longer U89.3
- net PAN5V.CS_3_P10: now also U95.1; no longer U95.3
- net PAN5V.CS_3_P11: now also U101.1; no longer U101.3
- net PAN5V.CS_3_P12: now also U107.1; no longer U107.3
- net PAN5V.CS_4_P02: now also U48.3; no longer U48.1
- net PAN5V.CS_4_P03: now also U54.3; no longer U54.1
- net PAN5V.CS_4_P04: now also U60.3; no longer U60.1
- net PAN5V.CS_4_P05: now also U66.3; no longer U66.1
- net PAN5V.CS_4_P06: now also U72.3; no longer U72.1
- net PAN5V.CS_4_P07: now also U78.3; no longer U78.1
- net PAN5V.CS_4_P08: now also U84.3; no longer U84.1
- net PAN5V.CS_4_P09: now also U90.3; no longer U90.1
- net PAN5V.CS_4_P10: now also U96.3; no longer U96.1
- net PAN5V.CS_4_P11: now also U102.3; no longer U102.1
- net PAN5V.CS_4_P12: now also U108.3; no longer U108.1
- net PAN5V.CS_5_P02: now also U48.1; no longer U48.3
- net PAN5V.CS_5_P03: now also U54.1; no longer U54.3
- net PAN5V.CS_5_P04: now also U60.1; no longer U60.3
- net PAN5V.CS_5_P05: now also U66.1; no longer U66.3
- net PAN5V.CS_5_P06: now also U72.1; no longer U72.3
- net PAN5V.CS_5_P07: now also U78.1; no longer U78.3
- net PAN5V.CS_5_P08: now also U84.1; no longer U84.3
- net PAN5V.CS_5_P09: now also U90.1; no longer U90.3
- net PAN5V.CS_5_P10: now also U96.1; no longer U96.3
- net PAN5V.CS_5_P11: now also U102.1; no longer U102.3
- net PAN5V.CS_5_P12: now also U108.1; no longer U108.3
- net PAN5V.CS_6_P02: now also U49.3; no longer U49.1
- net PAN5V.CS_6_P03: now also U55.3; no longer U55.1
- net PAN5V.CS_6_P04: now also U61.3; no longer U61.1
- net PAN5V.CS_6_P05: now also U67.3; no longer U67.1
- net PAN5V.CS_6_P06: now also U73.3; no longer U73.1
- net PAN5V.CS_6_P07: now also U79.3; no longer U79.1
- net PAN5V.CS_6_P08: now also U85.3; no longer U85.1
- net PAN5V.CS_6_P09: now also U91.3; no longer U91.1
- net PAN5V.CS_6_P10: now also U97.3; no longer U97.1
- net PAN5V.CS_6_P11: now also U103.3; no longer U103.1
- net PAN5V.CS_6_P12: now also U109.3; no longer U109.1
- net PAN5V.CS_7_P02: now also U49.1; no longer U49.3
- net PAN5V.CS_7_P03: now also U55.1; no longer U55.3
- net PAN5V.CS_7_P04: now also U61.1; no longer U61.3
- net PAN5V.CS_7_P05: now also U67.1; no longer U67.3
- net PAN5V.CS_7_P06: now also U73.1; no longer U73.3
- net PAN5V.CS_7_P07: now also U79.1; no longer U79.3
- net PAN5V.CS_7_P08: now also U85.1; no longer U85.3
- net PAN5V.CS_7_P09: now also U91.1; no longer U91.3
- net PAN5V.CS_7_P10: now also U97.1; no longer U97.3
- net PAN5V.CS_7_P11: now also U103.1; no longer U103.3
- net PAN5V.CS_7_P12: now also U109.1; no longer U109.3
- net PAN5V.EXT_INT: now also U104.3, U110.3, U50.3, U56.3, U62.3, U68.3, U74.3, U80.3, U86.3, U92.3, U98.3; no longer U104.1, U110.1, U50.1, U56.1, U62.1, U68.1, U74.1, U80.1, U86.1, U92.1, U98.1
- net PAN5V.MOSI_01: now also U45.1; no longer U45.3
- net PAN5V.MOSI_02: now also U51.1; no longer U51.3
- net PAN5V.MOSI_03: now also U57.1; no longer U57.3
- net PAN5V.MOSI_04: now also U63.1; no longer U63.3
- net PAN5V.MOSI_05: now also U69.1; no longer U69.3
- net PAN5V.MOSI_06: now also U75.1; no longer U75.3
- net PAN5V.MOSI_07: now also U81.1; no longer U81.3
- net PAN5V.MOSI_08: now also U87.1; no longer U87.3
- net PAN5V.MOSI_09: now also U93.1; no longer U93.3
- net PAN5V.MOSI_10: now also U99.1; no longer U99.3
- net PAN5V.MOSI_11: now also U105.1; no longer U105.3
- net PAN5V.SCK_0_H2: now also U75.3; no longer U75.1
- net PAN5V.SCK_1_H1: now also U45.3; no longer U45.1
- net PAN5V.SCK_1_H2: now also U81.3; no longer U81.1
- net PAN5V.SCK_2_H1: now also U51.3; no longer U51.1
- net PAN5V.SCK_2_H2: now also U87.3; no longer U87.1
- net PAN5V.SCK_3_H1: now also U57.3; no longer U57.1
- net PAN5V.SCK_3_H2: now also U93.3; no longer U93.1
- net PAN5V.SCK_4_H1: now also U63.3; no longer U63.1
- net PAN5V.SCK_4_H2: now also U99.3; no longer U99.1
- net PAN5V.SCK_5_H1: now also U69.3; no longer U69.1
- net PAN5V.SCK_5_H2: now also U105.3; no longer U105.1
- net at U71.4: now also R228.1; no longer R229.1
- net at U54.6: now also R195.1; no longer R194.1
- net at R287.1: now also U100.6; no longer U100.4
- net at R268.1: now also U91.4; no longer U91.6
- net at R247.1: now also U81.4; no longer U81.6
- net at R245.1: now also U79.6; no longer U79.4
- net at U76.6: now also R239.1; no longer R238.1
- net at R256.1: now also U85.4; no longer U85.6
- net at R304.1: now also U109.4; no longer U109.6
- net at R196.1: now also U55.4; no longer U55.6
- net at U96.4: now also R278.1; no longer R279.1
- net at R208.1: now also U61.4; no longer U61.6
- net at R265.1: now also U89.6; no longer U89.4
- net at U45.4: now also R175.1; no longer R176.1
- net at U60.6: now also R207.1; no longer R206.1
- net at U104.6: no longer R294.1
- net at R184.1: now also U49.4; no longer U49.6
- net at U53.4: now also R192.1; no longer R193.1
- net at R257.1: now also U85.6; no longer U85.4
- net at U56.4: now also R198.1
- net at U57.6: now also R200.1; no longer R199.1
- net at R217.1: now also U65.6; no longer U65.4
- net at U51.6: now also R188.1; no longer R187.1
- net at R212.1: now also U63.6; no longer U63.4
- net at U50.4: now also R186.1
- net at R255.1: now also U84.6; no longer U84.4
- net at R210.1: now also U62.4; no longer U62.6
- net at U59.4: now also R204.1; no longer R205.1
- net at U82.6: now also R251.1; no longer R250.1
- net at R281.1: now also U97.6; no longer U97.4
- net at R211.1: now also U63.4; no longer U63.6
- net at U107.4: now also R300.1; no longer R301.1
- net at U90.6: now also R267.1; no longer R266.1
- net at U46.6: now also R179.1; no longer R178.1
- net at U93.4: now also R271.1; no longer R272.1
- net at R246.1: now also U80.4; no longer U80.6
- net at U103.4: now also R292.1; no longer R293.1
- net at R226.1: now also U70.4; no longer U70.6
- net at R306.1: now also U110.4; no longer U110.6
- net at R264.1: now also U89.4; no longer U89.6
- net at U51.4: now also R187.1; no longer R188.1
- net at R280.1: now also U97.4; no longer U97.6
- net at R248.1: now also U81.6; no longer U81.4
- net at U64.4: now also R214.1; no longer R215.1
- net at U72.4: now also R230.1; no longer R231.1
- net at R263.1: now also U88.6; no longer U88.4
- net at U92.4: now also R270.1
- net at R243.1: now also U78.6; no longer U78.4
- net at U76.4: now also R238.1; no longer R239.1
- net at U73.4: now also R232.1; no longer R233.1
- net at R181.1: now also U47.6; no longer U47.4
- net at U75.4: now also R235.1; no longer R236.1
- net at U108.4: now also R302.1; no longer R303.1
- net at U107.6: now also R301.1; no longer R300.1
- net at R269.1: now also U91.6; no longer U91.4
- net at U54.4: now also R194.1; no longer R195.1
- net at U72.6: now also R231.1; no longer R230.1
- net at R185.1: now also U49.6; no longer U49.4
- net at U101.4: now also R288.1; no longer R289.1
- net at R262.1: now also U88.4; no longer U88.6
- net at U95.4: now also R276.1; no longer R277.1
- net at R286.1: now also U100.4; no longer U100.6
- net at R183.1: now also U48.6; no longer U48.4
- net at R244.1: now also U79.4; no longer U79.6
- net at R227.1: now also U70.6; no longer U70.4
- net at R197.1: now also U55.6; no longer U55.4
- net at U64.6: now also R215.1; no longer R214.1
- net at U99.6: now also R284.1; no longer R283.1
- net at U104.4: now also R294.1
- net at U96.6: now also R279.1; no longer R278.1
- net at U92.6: no longer R270.1
- net at R260.1: now also U87.6; no longer U87.4
- net at U58.4: now also R202.1; no longer R203.1
- net at R254.1: now also U84.4; no longer U84.6
- net at U52.6: now also R191.1; no longer R190.1
- net at U106.6: now also R299.1; no longer R298.1
- net at U98.4: now also R282.1
- net at U95.6: now also R277.1; no longer R276.1
- net at U66.6: now also R219.1; no longer R218.1
- net at U45.6: now also R176.1; no longer R175.1
- net at U90.4: now also R266.1; no longer R267.1
- net at R216.1: now also U65.4; no longer U65.6
- net at R180.1: now also U47.4; no longer U47.6
- net at U69.4: now also R223.1; no longer R224.1
- net at U69.6: now also R224.1; no longer R223.1
- net at U82.4: now also R250.1; no longer R251.1
- net at U59.6: now also R205.1; no longer R204.1
- net at U53.6: now also R193.1; no longer R192.1
- net at U71.6: now also R229.1; no longer R228.1
- net at U58.6: now also R203.1; no longer R202.1
- net at U52.4: now also R190.1; no longer R191.1
- net at R209.1: now also U61.6; no longer U61.4
- net at R258.1: now also U86.4; no longer U86.6
- net at U46.4: now also R178.1; no longer R179.1
- net at R291.1: now also U102.6; no longer U102.4
- net at U98.6: no longer R282.1
- net at U93.6: now also R272.1; no longer R271.1
- net at U60.4: now also R206.1; no longer R207.1
- net at U57.4: now also R199.1; no longer R200.1
- net at R259.1: now also U87.4; no longer U87.6
- net at U101.6: now also R289.1; no longer R288.1
- net at U68.4: now also R222.1
- net at U108.6: now also R303.1; no longer R302.1
- net at R234.1: now also U74.4; no longer U74.6
- net at R220.1: now also U67.4; no longer U67.6
- net at U56.6: no longer R198.1
- net at U105.6: now also R296.1; no longer R295.1
- net at R221.1: now also U67.6; no longer U67.4
- net at R182.1: now also U48.4; no longer U48.6
- net at U103.6: now also R293.1; no longer R292.1
- net at R242.1: now also U78.4; no longer U78.6
- net at R290.1: now also U102.4; no longer U102.6
- net at U83.6: now also R253.1; no longer R252.1
- net at U77.6: now also R241.1; no longer R240.1
- net at U77.4: now also R240.1; no longer R241.1
- net at U66.4: now also R218.1; no longer R219.1
- net at U99.4: now also R283.1; no longer R284.1
- net at U94.4: now also R274.1; no longer R275.1
- net at U75.6: now also R236.1; no longer R235.1
- net at U106.4: now also R298.1; no longer R299.1
- net at U73.6: now also R233.1; no longer R232.1
- net at U83.4: now also R252.1; no longer R253.1
- net at U105.4: now also R295.1; no longer R296.1
- net at U50.6: no longer R186.1
- net at U68.6: no longer R222.1
- net at R305.1: now also U109.6; no longer U109.4
- net at U94.6: now also R275.1; no longer R274.1
Other:
- moved on the sheet: U100A, U100B, U101A, U101B, U102A, U102B, U103A, U103B, U104A, U104B, U105A, U105B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
