File: development/arena_12-12/ni/ni_arena_12-12_v0p1/panel_headers.kicad_sch (KiCad schematic)
At the start: 315 parts, among them P1 CONN15, P10 CONN15, P11 CONN15, P12 CONN15, P2 CONN15, P3 CONN15, P4 CONN15, P5 CONN15, P6 CONN15, P7 CONN15, P8 CONN15, P9 CONN15, Q1 MOSFET_NCHAN, U100 74LVC2G17, U101 74LVC2G17, U102 74LVC2G17, U103 74LVC2G17, U104 74LVC2G17, U105 74LVC2G17, U106 74LVC2G17, U107 74LVC2G17, U108 74LVC2G17, U109 74LVC2G17, U110 74LVC2G17, U39 74LVC2G17, U40 74LVC2G17, U41 74LVC2G17, U42 74LVC2G17, U43 74LVC2G17, U44 74LVC2G17, U45 74LVC2G17, U46 74LVC2G17, U47 74LVC2G17, U48 74LVC2G17, U49 74LVC2G17, U50 74LVC2G17, U51 74LVC2G17, U52 74LVC2G17, U53 74LVC2G17, U54 74LVC2G17, U55 74LVC2G17, U56 74LVC2G17, U57 74LVC2G17, U58 74LVC2G17, U59 74LVC2G17, U60 74LVC2G17, U61 74LVC2G17, U62 74LVC2G17, U63 74LVC2G17, U64 74LVC2G17, U65 74LVC2G17, U66 74LVC2G17, U67 74LVC2G17, U68 74LVC2G17, U69 74LVC2G17, U70 74LVC2G17, U71 74LVC2G17, U72 74LVC2G17, U73 74LVC2G17, U74 74LVC2G17, U75 74LVC2G17, U76 74LVC2G17, U77 74LVC2G17, U78 74LVC2G17, U79 74LVC2G17, U80 74LVC2G17, U81 74LVC2G17, U82 74LVC2G17, U83 74LVC2G17, U84 74LVC2G17, U85 74LVC2G17, U86 74LVC2G17, U87 74LVC2G17, U88 74LVC2G17, U89 74LVC2G17, U90 74LVC2G17, U91 74LVC2G17, U92 74LVC2G17, U93 74LVC2G17, U94 74LVC2G17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

Commit message: Worked on fabrication setup for NI 12-12 arena.
Added part numbers, datasheets, etc. to symbol table.
Deleted old productions files.
Parts:
- C1, C10, C11, C12, C2, C3, C4, C5, C6, C7, C8, C9: LCSC Part # (none) -> C7432790; MPN (none) -> HGC1210R5107M160NSVK
- C100, C101, C102, C103, C104, C105, C106, C35, C36, C37, C38, C39, C40, C41, C42, C43, C44, C45, C46, C47, C48, C49, C50, C51, C52, C53, C54, C55, C56, C57, C58, C59, C60, C61, C62, C63, C64, C65, C66, C67, C68, C69, C70, C71, C72, C73, C74, C75, C76, C77, C78, C79, C80, C81, C82, C83, C84, C85, C86, C87, C88, C89, C90, C91, C92, C93, C94, C95, C96, C97, C98, C99: Digikey PN (none) -> 1276-1001-2-ND; LCSC Part # (none) -> C1525; MPN (none) -> CL05B104KO5NNNC
- P1, P10, P11, P12, P2, P3, P4, P5, P6, P7, P8, P9: Digikey PN (none) -> S7048-ND; LCSC Part # (none) -> C18078136; MPN (none) -> PPPC151LFBN-RC
- Q1: LCSC Part # (none) -> C165220; MPN (none) -> ME2306D
- R163, R164, R165, R166, R167, R168, R169, R170, R171, R172, R173, R174, R175, R176, R177, R178, R179, R180, R181, R182, R183, R184, R185, R186, R187, R188, R189, R190, R191, R192, R193, R194, R195, R196, R197, R198, R199, R200, R201, R202, R203, R204, R205, R206, R207, R208, R209, R210, R211, R212, R213, R214, R215, R216, R217, R218, R219, R220, R221, R222, R223, R224, R225, R226, R227, R228, R229, R230, R231, R232, R233, R234, R235, R236, R237, R238, R239, R240, R241, R242, R243, R244, R245, R246, R247, R248, R249, R250, R251, R252, R253, R254, R255, R256, R257, R258, R259, R260, R261, R262, R263, R264, R265, R266, R267, R268, R269, R270, R271, R272, R273, R274, R275, R276, R277, R278, R279, R280, R281, R282, R283, R284, R285, R286, R287, R288, R289, R290, R291, R292, R293, R294, R295, R296, R297, R298, R299, R300, R301, R302, R303, R304, R305, R306: Digikey PN (none) -> (none); LCSC Part # (none) -> C25105; MPN (none) -> 0402WGF330JTCE
- R307: LCSC Part # (none) -> C25765; MPN (none) -> 0402WGF2002TCE
- R308: LCSC Part # (none) -> C25087; MPN (none) -> 0402WGF2000TCE
- U100, U101, U102, U103, U104, U105, U106, U107, U108, U109, U110, U39, U40, U41, U42, U43, U44, U45, U46, U47, U48, U49, U50, U51, U52, U53, U54, U55, U56, U57, U58, U59, U60, U61, U62, U63, U64, U65, U66, U67, U68, U69, U70, U71, U72, U73, U74, U75, U76, U77, U78, U79, U80, U81, U82, U83, U84, U85, U86, U87, U88, U89, U90, U91, U92, U93, U94, U95, U96, U97, U98, U99: Digikey PN (none) -> 296-SN74LVC2G17DBVRTR-ND; LCSC Part # (none) -> C10429; MPN (none) -> SN74LVC2G17DBVR

Commit message: Finished preliminary production setup for NI 12-12 arena with schmitt buffers.
Note,  rotation offsets may still adjusting (for 74LVC2G17's and Q1)
Parts:
- Q1, U100, U101, U102, U103, U104, U105, U106, U107, U108, U109, U110, U39, U40, U41, U42, U43, U44, U45, U46, U47, U48, U49, U50, U51, U52, U53, U54, U55, U56, U57, U58, U59, U60, U61, U62, U63, U64, U65, U66, U67, U68, U69, U70, U71, U72, U73, U74, U75, U76, U77, U78, U79, U80, U81, U82, U83, U84, U85, U86, U87, U88, U89, U90, U91, U92, U93, U94, U95, U96, U97, U98, U99: FT Rotation Offset (none) -> 0

Commit message: project cleanup prior to ordering
Other:
- company: (none) -> IORodeo for Reiserlab @ Janelia
- title: (none) -> 12-12 NI G4.1 Arena Modular LED Display
Changed lines of the file:
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@@
 	(generator_version "9.0")
 	(paper "User" 1016 812.8)
+	(title_block
+		(title "12-12 NI G4.1 Arena Modular LED Display")
+		(date "2025-04-21")
+		(rev "v0.3.4")
+		(company "IORodeo for Reiserlab @ Janelia")
+	)
 	(text "Panel base capacitor: C7432790 16V 100uF"
 		(exclude_from_sim no)
