File: development/arena_12-12/ni/ni_arena_12-12_v0p1/level_shifters.kicad_sch (KiCad schematic)
At the start: 225 parts, among them U10 TXB0108PW, U11 TXB0108PW, U12 TXB0108PW, U13 TXB0108PW, U14 TXB0108PW, U15 TXB0108PW, U16 TXB0108PW, U17 TXB0108PW, U18 TXB0108PW, U19 74LVC2G17, U2 TXB0108PW, U20 74LVC2G17, U21 74LVC2G17, U22 74LVC2G17, U23 74LVC2G17, U24 74LVC2G17, U25 74LVC2G17, U26 74LVC2G17, U27 74LVC2G17, U28 74LVC2G17, U29 74LVC2G17, U3 TXB0108PW, U30 74LVC2G17, U31 74LVC2G17, U32 74LVC2G17, U33 74LVC2G17, U34 74LVC2G17, U35 74LVC2G17, U36 74LVC2G17, U37 74LVC2G17, U38 74LVC2G17, U4 TXB0108PW, U5 TXB0108PW, U6 TXB0108PW, U7 TXB0108PW, U8 TXB0108PW, U9 TXB0108PW

Commit message: Worked on fabrication setup for NI 12-12 arena.
Added part numbers, datasheets, etc. to symbol table.
Deleted old productions files.
Parts:
- C107, C108, C109, C110, C111, C112, C113, C114, C115, C116, C117, C118, C119, C120, C121, C122, C123, C124, C125, C126, C127, C128, C129, C130, C131, C132, C133, C134, C135, C136, C137, C138, C139, C140, C15, C16, C17, C18, C19, C20, C21, C22, C23, C24, C25, C26, C27, C28, C29, C30, C31, C32, C33, C34: Digikey PN (none) -> 1276-1001-2-ND; LCSC Part # (none) -> C1525; MPN (none) -> CL05B104KO5NNNC
- R100, R101, R102, R103, R104, R105, R106, R107, R108, R109, R110, R111, R112, R113, R114, R115, R116, R117, R118, R119, R120, R121, R122, R123, R124, R125, R126, R127, R128, R129, R130, R131, R132, R133, R134, R135, R136, R137, R138, R139, R140, R141, R142, R143, R144, R145, R146, R147, R148, R149, R150, R151, R152, R153, R154, R155, R156, R157, R158, R159, R160, R161, R162, R29, R30, R31, R32, R33, R34, R35, R36, R37, R38, R39, R40, R41, R42, R43, R44, R45, R46, R47, R48, R49, R50, R51, R52, R53, R54, R55, R56, R57, R58, R59, R60, R61, R62, R63, R64, R65, R66, R67, R68, R69, R70, R71, R72, R73, R74, R75, R76, R77, R78, R79, R80, R81, R82, R83, R84, R85, R86, R87, R88, R89, R90, R91, R92, R93, R94, R95, R96, R97, R98, R99: Digikey PN (none) -> (none); LCSC Part # (none) -> C25105; MPN (none) -> 0402WGF330JTCE
- U10, U11, U12, U13, U14, U15, U16, U17, U18, U2, U3, U4, U5, U6, U7, U8, U9: Digikey PN (none) -> 296-21527-2-ND; LCSC Part # (none) -> C53406; MPN (none) -> TXB0108PWR
- U19, U20, U21, U22, U23, U24, U25, U26, U27, U28, U29, U30, U31, U32, U33, U34, U35, U36, U37, U38: Digikey PN (none) -> 296-SN74LVC2G17DBVRTR-ND; LCSC Part # (none) -> C10429; MPN (none) -> SN74LVC2G17DBVR

Commit message: Finished preliminary production setup for NI 12-12 arena with schmitt buffers.
Note,  rotation offsets may still adjusting (for 74LVC2G17's and Q1)
Parts:
- U19, U20, U21, U22, U23, U24, U25, U26, U27, U28, U29, U30, U31, U32, U33, U34, U35, U36, U37, U38: FT Rotation Offset (none) -> 0

Commit message: project cleanup prior to ordering
Other:
- company: (none) -> IORodeo for Reiserlab @ Janelia
- title: (none) -> 12-12 NI G4.1 Arena Modular LED Display
Changed lines of the file:
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@@
 	(generator_version "9.0")
 	(paper "User" 711.2 711.2)
+	(title_block
+		(title "12-12 NI G4.1 Arena Modular LED Display")
+		(date "2025-04-21")
+		(rev "v0.3.4")
+		(company "IORodeo for Reiserlab @ Janelia")
+	)
 	(bus_alias "PAN5V"
 		(members "CS_0_P01" "CS_0_P02" "CS_0_P03" "CS_0_P04" "CS_0_P05" "CS_0_P06"
