File: development/arena_12-12/ni/ni_arena_12-12_v0p1/ni_arena_12-12.kicad_sch (KiCad schematic)
At the start: 0 parts

Commit message: project cleanup prior to ordering
Other:
- company: (none) -> IORodeo for Reiserlab @ Janelia
- title: (none) -> 12-12 NI G4.1 Arena Modular LED Display
Changed lines of the file:
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@@
 	(paper "User" 279.4 203.2)
 	(title_block
-		(date "11 jun 2015")
+		(title "12-12 NI G4.1 Arena Modular LED Display")
+		(date "2025-04-21")
+		(rev "v0.3.4")
+		(company "IORodeo for Reiserlab @ Janelia")
 	)
 	(text "12-12 NI Arena"
