File: development/arena_12-12/ni/ni_arena_12-12_v0p1/power.kicad_sch (KiCad schematic)
At the start: 6 parts, among them J1 Barrel_Jack, J3 Barrel_Jack, SW1 SW_SPDT, U1 AP2112K-3.3

Commit message: Worked on fabrication setup for NI 12-12 arena.
Added part numbers, datasheets, etc. to symbol table.
Deleted old productions files.
Parts:
- C13, C14: LCSC Part # (none) -> C342827; MPN (none) -> C3216X7R1C106KT000N
- J1, J3: Digikey PN (none) -> CP-063AH-ND; LCSC Part # (none) -> C2928097; MPN (none) -> PJ-063AH
- SW1: Digikey PN (none) -> CKC5102-ND; LCSC Part # (none) -> C2798743; MPN (none) -> L102021ML04Q
- U1: Digikey PN (none) -> AP2112K-3.3TRG1DICT-ND; LCSC Part # (none) -> C51118; MPN (none) -> AP2112K-3.3TRG1
Changed lines of the file:
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@@
 			)
 		)
-		(property "Datasheet" "~"
+		(property "Datasheet" "https://www.lcsc.com/datasheet/lcsc_datasheet_2410121551_TDK-C3216X7R1C106KT000N_C342827.pdf"
 			(at 199.39 72.39 0)
 			(effects
@@
 		)
 		(property "Description" ""
+			(at 199.39 72.39 0)
+			(effects
+				(font
+					(size 1.27 1.27)
+				)
+				(hide yes)
+			)
+		)
+		(property "LCSC Part #" "C342827"
+			(at 199.39 72.39 0)
+			(effects
+				(font
+					(size 1.27 1.27)
+				)
+				(hide yes)
+			)
+		)
+		(property "MPN" "C3216X7R1C106KT000N "
 			(at 199.39 72.39 0)
 			(effects
@@
 			)
 		)
-		(property "Datasheet" "~"
+		(property "Datasheet" "https://datasheet.octopart.com/PJ-063AH-Same-Sky-datasheet-181917378.pdf"
 			(at 99.06 65.532 0)
 			(effects
@@
 		)
 		(property "Description" ""
+			(at 100.33 64.516 0)
+			(effects
+				(font
+					(size 1.27 1.27)
+				)
+				(hide yes)
+			)
+		)
+		(property "Digikey PN" "CP-063AH-ND"
+			(at 100.33 64.516 0)
+			(effects
+				(font
+					(size 1.27 1.27)
+				)
+				(hide yes)
+			)
+		)
+		(property "LCSC Part #" "C2928097"
+			(at 100.33 64.516 0)
+			(effects
+				(font
+					(size 1.27 1.27)
+				)
+				(hide yes)
+			)
+		)
+		(property "MPN" "PJ-063AH"
 			(at 100.33 64.516 0)
 			(effects
@@
 			)
 		)
-		(property "Datasheet" "~"
+		(property "Datasheet" "https://datasheet.octopart.com/L102021ML04Q-C%26K-Components-datasheet-62111167.pdf"
 			(at 67.31 64.516 0)
 			(effects
@@
 		)
 		(property "Description" ""
+			(at 67.31 64.516 0)
+			(effects
+				(font
+					(size 1.27 1.27)
+				)
+				(hide yes)
+			)
+		)
+		(property "Digikey PN" "CKC5102-ND"
+			(at 67.31 64.516 0)
+			(effects
+				(font
+					(size 1.27 1.27)
+				)
+				(hide yes)
+			)
+		)
+		(property "LCSC Part #" "C2798743"
+			(at 67.31 64.516 0)
+			(effects
+				(font
+					(size 1.27 1.27)
+				)
+				(hide yes)
+			)
+		)
+		(property "MPN" "L102021ML04Q"
 			(at 67.31 64.516 0)
 			(effects
@@
 			)
 		)
-		(property "Datasheet" "~"
+		(property "Datasheet" "https://datasheet.octopart.com/PJ-063AH-Same-Sky-datasheet-181917378.pdf"
 			(at 100.33 87.376 0)
 			(effects
@@
 		)
 		(property "Description" ""
+			(at 101.6 86.36 0)
+			(effects
+				(font
+					(size 1.27 1.27)
+				)
+				(hide yes)
+			)
+		)
+		(property "Digikey PN" "CP-063AH-ND"
+			(at 101.6 86.36 0)
+			(effects
+				(font
+					(size 1.27 1.27)
+				)
+				(hide yes)
+			)
+		)
+		(property "LCSC Part #" "C2928097"
+			(at 101.6 86.36 0)
+			(effects
+				(font
+					(size 1.27 1.27)
+				)
+				(hide yes)
+			)
+		)
+		(property "MPN" "PJ-063AH"
 			(at 101.6 86.36 0)
 			(effects
@@
 			)
 		)
-		(property "Datasheet" "~"
+		(property "Datasheet" "https://www.lcsc.com/datasheet/lcsc_datasheet_2410121551_TDK-C3216X7R1C106KT000N_C342827.pdf"
 			(at 168.91 72.39 0)
 			(effects
@@
 		)
 		(property "Description" ""
+			(at 168.91 72.39 0)
+			(effects
+				(font
+					(size 1.27 1.27)
+				)
+				(hide yes)
+			)
+		)
+		(property "LCSC Part #" "C342827"
+			(at 168.91 72.39 0)
+			(effects
+				(font
+					(size 1.27 1.27)
+				)
+				(hide yes)
+			)
+		)
+		(property "MPN" "C3216X7R1C106KT000N "
 			(at 168.91 72.39 0)
 			(effects
@@
 			(at 187.96 67.31 0)
 			(effects
+				(font
+					(size 1.27 1.27)
+				)
+				(hide yes)
+			)
+		)
+		(property "Digikey PN" "AP2112K-3.3TRG1DICT-ND"
+			(at 187.96 67.31 0)
+			(effects
+				(font
+					(size 1.27 1.27)
+				)
+				(hide yes)
+			)
+		)
+		(property "LCSC Part #" "C51118"
+			(at 187.96 67.31 0)
+			(effects
+				(font
+					(size 1.27 1.27)
+				)
+				(hide yes)
+			)
+		)
+		(property "MPN" "AP2112K-3.3TRG1"
+			(at 187.96 67.31 0)
+			(effects

Commit message: project cleanup prior to ordering
Other:
- company: (none) -> IORodeo for Reiserlab @ Janelia
- title: (none) -> 12-12 NI G4.1 Arena Modular LED Display
Changed lines of the file:
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@@
 	(generator_version "9.0")
 	(paper "A4")
+	(title_block
+		(title "12-12 NI G4.1 Arena Modular LED Display")
+		(date "2025-04-21")
+		(rev "v0.3.4")
+		(company "IORodeo for Reiserlab @ Janelia")
+	)
 	(text "5V"
 		(exclude_from_sim no)
