File: arena_12-12/arena_12-12_G4.1_belt/panel_headers.kicad_sch (KiCad schematic)
At the start: 36 parts, among them P1 CONN15, P10 CONN15, P11 CONN15, P12 CONN15, P2 CONN15, P3 CONN15, P4 CONN15, P5 CONN15, P6 CONN15, P7 CONN15, P8 CONN15, P9 CONN15

Commit message: cleanup, belt with SMD power connector
Other:
- title: 12-12 Teensy G4.1 Arena Belt Modular LED Display -> Arena 12-12 G4.1 Belt :: Modular LED Display
Changed lines of the file:
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@@
 	(paper "User" 304.8 508)
 	(title_block
-		(title "12-12 Teensy G4.1 Arena Belt Modular LED Display")
-		(date "2025-07-22")
-		(rev "v0.5.1")
+		(title "Arena 12-12 G4.1 Belt :: Modular LED Display")
+		(date "2025-07-24")
+		(rev "v0.1")
 		(company "MCN-NET @ Janelia")
 	)
@@
 		(effects
 			(font
+				(face "KiCad Font")
 				(size 5.08 5.08)
 				(thickness 0.508)
