File: arena_12-12/arena_12-12_G4.1_belt/arena_12-12_G4.1_belt.kicad_pcb (KiCad board)
At the start: 2 copper layers, 228.6 x 228.6 mm, 41 parts, among them J4 Barrel_Jack, P1 CONN15, P10 CONN15, P11 CONN15, P12 CONN15, P2 CONN15, P3 CONN15, P4 CONN15, P5 CONN15, P6 CONN15, P7 CONN15, P8 CONN15, P9 CONN15

Commit message: fix issues, bump to top-0.4.3 and belt-0.2
Routing:
- net +5V: track 136.3 -> 157.0 mm, vias 2 -> 10
Changed lines of the file:
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@@
 	(title_block
 		(title "Arena 12-12 G4.1 Belt :: Modular LED Display")
-		(date "2025-07-24")
-		(rev "v0.1")
+		(date "2025-07-25")
+		(rev "v0.2")
 		(company "MCN-NET @ Janelia")
 	)
@@
 	)
 	(gr_text "5V\n"
-		(at 93.8 85.19 180)
+		(at 94.25 85.75 180)
 		(layer "B.SilkS")
 		(effects
@@
 	)
 	(via
+		(at 95 84.75)
+		(size 0.6)
+		(drill 0.3)
+		(layers "F.Cu" "B.Cu")
+		(free yes)
+		(net 1)
+	)
+	(via
+		(at 92.75 86)
+		(size 0.6)
+		(drill 0.3)
+		(layers "F.Cu" "B.Cu")
+		(free yes)
+		(net 1)
+	)
+	(via
 		(at 99.7 86)
 		(size 0.6)
@@
 	)
 	(via
+		(at 96 84.75)
+		(size 0.6)
+		(drill 0.3)
+		(layers "F.Cu" "B.Cu")
+		(free yes)
+		(net 1)
+	)
+	(via
+		(at 94 85)
+		(size 0.6)
+		(drill 0.3)
+		(layers "F.Cu" "B.Cu")
+		(free yes)
+		(net 1)
+	)
+	(via
+		(at 97 84.75)
+		(size 0.6)
+		(drill 0.3)
+		(layers "F.Cu" "B.Cu")
+		(free yes)
+		(net 1)
+	)
+	(via
+		(at 98.5 86)
+		(size 0.6)
+		(drill 0.3)
+		(layers "F.Cu" "B.Cu")
+		(free yes)
+		(net 1)
+	)
+	(via
+		(at 93.75 86)
+		(size 0.6)
+		(drill 0.3)
+		(layers "F.Cu" "B.Cu")
+		(free yes)
+		(net 1)
+	)
+	(via
 		(at 91.7 86)
 		(size 0.6)
@@
 		(net 1)
 	)
+	(via
+		(at 97.75 85.25)
+		(size 0.6)
+		(drill 0.3)
+		(layers "F.Cu" "B.Cu")
+		(free yes)
+		(net 1)
+	)
 	(segment
 		(start 279.348017 215.630078)
@@
 	)
 	(segment
+		(start 97.75 85.25)
+		(end 98.5 86)
+		(width 0.8)
+		(layer "B.Cu")
+		(net 1)
+	)
+	(segment
 		(start 246.828122 261.335817)
 		(end 250.934764 258.99224)
@@
 	)
 	(segment
+		(start 95 84.75)
+		(end 96 84.75)
+		(width 0.8)
+		(layer "B.Cu")
+		(net 1)
+	)
+	(segment
 		(start 256.598561 111.775053)
 		(end 261.335817 108.771877)
@@
 	)
 	(segment
+		(start 93.75 86)
+		(end 94 85)
+		(width 0.8)
+		(layer "B.Cu")
+		(net 1)
+	)
+	(segment
 		(start 99.001438 243.824946)
 		(end 94.264182 246.828122)
@@
 	)
 	(segment
+		(start 97.75 85.25)
+		(end 95.7 81.44)
+		(width 0.8)
+		(layer "B.Cu")
+		(net 1)
+	)
+	(segment
 		(start 91.7 86)
 		(end 95.7 81.44)
@@
 	)
 	(segment
+		(start 96 84.75)
+		(end 97 84.75)
+		(width 0.8)
+		(layer "B.Cu")
+		(net 1)
+	)
+	(segment
+		(start 91.7 86)
+		(end 92.75 86)
+		(width 0.8)
+		(layer "B.Cu")
+		(net 1)
+	)
+	(segment
+		(start 94 85)
+		(end 95.7 81.44)
+		(width 0.8)
+		(layer "B.Cu")
+		(net 1)
+	)
+	(segment
 		(start 261.335817 108.771877)
 		(end 258.99224 104.665235)
@@
 	)
 	(segment
+		(start 97 84.75)
+		(end 97.75 85.25)
+		(width 0.8)
+		(layer "B.Cu")
+		(net 1)
+	)
+	(segment
+		(start 92.75 86)
+		(end 93.75 86)
+		(width 0.8)
+		(layer "B.Cu")
+		(net 1)
+	)
+	(segment
 		(start 274.378561 213.029082)
 		(end 279.348017 215.630078)
@@
 	)
 	(segment
+		(start 98.5 86)
+		(end 99.7 86)
+		(width 0.8)
+		(layer "B.Cu")
+		(net 1)
+	)
+	(segment
+		(start 94 85)
+		(end 95 84.75)
+		(width 0.8)
+		(layer "B.Cu")
+		(net 1)
+	)
+	(segment
 		(start 76.545971 195.58)
 		(end 70.941799 195.8122)
@@
 	)
 	(segment
+		(start 96 84.75)
+		(end 95.7 81.44)
+		(width 0.8)
+		(layer "B.Cu")
+		(net 1)
+	)
+	(segment
 		(start 81.221438 142.570917)
 		(end 76.251982 139.969921)
@@
 		(width 0.8)
 		(layer "B.Cu")
-		(net 1)
-	)
-	(segment
-		(start 89.125971 195.58)
-		(end 89.19 195.51)
-		(width 0.8)
-		(layer "B.Cu")
