File: arena_12-12/arena_12-12_G4.1_top/arena_top_12-12.kicad_pcb (KiCad board)
At the start: 2 copper layers, 228.6 x 228.6 mm, 41 parts, among them J4 Barrel_Jack, P1 CONN15, P10 CONN15, P11 CONN15, P12 CONN15, P2 CONN15, P3 CONN15, P4 CONN15, P5 CONN15, P6 CONN15, P7 CONN15, P8 CONN15, P9 CONN15

Commit message: fix issues, bump to top-0.4.3 and belt-0.2
Routing:
- net +5V: track 129.1 -> 178.3 mm, vias 1 -> 9
