File: arena_12-12/arena_12-12_G4.1_top/arena_top_12-12.kicad_sch (KiCad schematic)
At the start: 0 parts

Commit message: bump version
Other:
- company: (none) -> IORodeo for Reiserlab @ Janelia
- title: (none) -> 12-12 Teensy G4.1 Arena Top Modular LED Display
Changed lines of the file:
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@@
 (kicad_sch
-	(version 20231120)
+	(version 20250114)
 	(generator "eeschema")
-	(generator_version "8.0")
+	(generator_version "9.0")
 	(paper "User" 279.4 203.2)
 	(title_block
-		(date "11 jun 2015")
+		(title "12-12 Teensy G4.1 Arena Top Modular LED Display")
+		(date "2025-07-22")
+		(rev "v0.4")
+		(company "IORodeo for Reiserlab @ Janelia")
 	)
 	(text "12-12 Teensy Arena Top"
@@
 		(at 106.68 48.26)
 		(size 27.432 18.161)
+		(exclude_from_sim no)
+		(in_bom yes)
+		(on_board yes)
+		(dnp no)
 		(fields_autoplaced yes)
 		(stroke
@@
 		(at 141.986 48.768)
 		(size 30.226 18.034)
+		(exclude_from_sim no)
+		(in_bom yes)
+		(on_board yes)
+		(dnp no)
 		(fields_autoplaced yes)
 		(stroke
@@
 		(at 67.31 48.26)
 		(size 30.48 18.161)
+		(exclude_from_sim no)
+		(in_bom yes)
+		(on_board yes)
+		(dnp no)
 		(fields_autoplaced yes)
 		(stroke
@@
 		)
 	)
+	(embedded_fonts no)
 )

Commit message: cleanup top, v0.4.2
Other:
- note added: "Arena Top 12-12"
- note removed: "12-12 Teensy Arena Top"
- title: 12-12 Teensy G4.1 Arena Top Modular LED Display -> G4.1 Arena Top :: Modular LED Display
Changed lines of the file:
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@@
 	(paper "User" 279.4 203.2)
 	(title_block
-		(title "12-12 Teensy G4.1 Arena Top Modular LED Display")
-		(date "2025-07-22")
-		(rev "v0.4.1")
+		(title "G4.1 Arena Top :: Modular LED Display")
+		(date "2025-07-24")
+		(rev "v0.4.2")
 		(company "IORodeo for Reiserlab @ Janelia")
 	)
-	(text "12-12 Teensy Arena Top"
+	(text "Arena Top 12-12"
 		(exclude_from_sim no)
 		(at 90.678 30.734 0)
@@
 			(font
 				(size 5.08 5.08)
+				(thickness 1.016)
+				(bold yes)
 			)
 			(justify left bottom)
