File: arena_12-12/arena_12-12_G4.1_top/holes.kicad_sch (KiCad schematic)
At the start: 4 parts

Commit message: bump version
Parts:
- H1, H2, H3, H4: now left out of the parts list
Changed lines of the file:
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@@
 (kicad_sch
-	(version 20231120)
+	(version 20250114)
 	(generator "eeschema")
-	(generator_version "8.0")
+	(generator_version "9.0")
 	(paper "A4")
 	(title_block
 		(title "12-12 Teensy G4.1 Arena Top Modular LED Display")
-		(date "2024-12-23")
-		(rev "v0.3")
+		(date "2025-07-22")
+		(rev "v0.4")
 		(company "IORodeo for Reiserlab @ Janelia")
 	)
@@
 	(label "Ground Holes"
 		(at 125.73 33.02 0)
-		(fields_autoplaced yes)
 		(effects
 			(font
@@
 		(unit 1)
 		(exclude_from_sim no)
-		(in_bom yes)
+		(in_bom no)
 		(on_board yes)
 		(dnp yes)
@@
 		(unit 1)
 		(exclude_from_sim no)
-		(in_bom yes)
+		(in_bom no)
 		(on_board yes)
 		(dnp yes)
@@
 		(unit 1)
 		(exclude_from_sim no)
-		(in_bom yes)
+		(in_bom no)
 		(on_board yes)
 		(dnp yes)
@@
 		(unit 1)
 		(exclude_from_sim no)
-		(in_bom yes)
+		(in_bom no)
 		(on_board yes)
 		(dnp yes)

Commit message: cleanup top, v0.4.2
Other:
- note added: "Ground Holes"
- title: 12-12 Teensy G4.1 Arena Top Modular LED Display -> G4.1 Arena Top :: Modular LED Display
Changed lines of the file:
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@@
 	(paper "A4")
 	(title_block
-		(title "12-12 Teensy G4.1 Arena Top Modular LED Display")
-		(date "2025-07-22")
-		(rev "v0.4.1")
+		(title "G4.1 Arena Top :: Modular LED Display")
+		(date "2025-07-24")
+		(rev "v0.4.2")
 		(company "IORodeo for Reiserlab @ Janelia")
+	)
+	(text "Ground Holes"
+		(exclude_from_sim no)
+		(at 140.462 26.162 0)
+		(effects
+			(font
+				(size 5.08 5.08)
+				(thickness 1.016)
+				(bold yes)
+			)
+		)
 	)
 	(wire
@@
 		)
 	)
-	(label "Ground Holes"
-		(at 125.73 33.02 0)
-		(effects
-			(font
-				(size 5.08 5.08)
-				(thickness 1.016)
-				(bold yes)
-			)
-			(justify left bottom)
-		)
-	)
