File: arena_12-12/arena_12-12_G4.1_top/panel_headers.kicad_sch (KiCad schematic)
At the start: 36 parts, among them P1 CONN15, P10 CONN15, P11 CONN15, P12 CONN15, P2 CONN15, P3 CONN15, P4 CONN15, P5 CONN15, P6 CONN15, P7 CONN15, P8 CONN15, P9 CONN15

Commit message: One-sided version
Parts:
- C13, C14, C15, C16, C17, C18, C19, C20, C21, C22, C23, C24: footprint Capacitor_THT:CP_Radial_D8.0mm_P2.50mm -> Capacitor_SMD:CP_Elec_6.3x7.7; DigiKey PN 1189-1856-ND -> PCE5024TR-ND; LCSC Part # C338173 -> C165974; MPN 16YXF100MEFC6.3X11 -> EEEFTH101XAP
Changed lines of the file:
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@@
 		(title "12-12 Teensy G4.1 Arena Top Modular LED Display")
 		(date "2025-07-22")
-		(rev "v0.4")
+		(rev "v0.4.1")
 		(company "IORodeo for Reiserlab @ Janelia")
 	)
@@
 			)
 		)
-		(property "Footprint" "Capacitor_THT:CP_Radial_D8.0mm_P2.50mm"
+		(property "Footprint" "Capacitor_SMD:CP_Elec_6.3x7.7"
 			(at 56.8452 80.01 0)
 			(effects
@@
 			)
 		)
-		(property "Datasheet" "https://octopart.com/datasheet/16yxf100mefc6.3x11-rubycon-19941780"
+		(property "Datasheet" "https://octopart.com/datasheet/eeefth101xap-panasonic-19787188"
 			(at 55.88 76.2 0)
 			(effects
@@
 			)
 		)
-		(property "DigiKey PN" "1189-1856-ND"
+		(property "DigiKey PN" "PCE5024TR-ND"
 			(at 55.88 76.2 0)
 			(effects
@@
 			)
 		)
-		(property "LCSC Part #" " C338173"
+		(property "LCSC Part #" "C165974"
 			(at 55.88 76.2 0)
 			(effects
@@
 			)
 		)
-		(property "MPN" "16YXF100MEFC6.3X11"
+		(property "MPN" "EEEFTH101XAP"
 			(at 55.88 76.2 0)
 			(effects
@@
 			)
 		)
-		(property "Footprint" "Capacitor_THT:CP_Radial_D8.0mm_P2.50mm"
+		(property "Footprint" "Capacitor_SMD:CP_Elec_6.3x7.7"
 			(at 56.8452 204.47 0)
 			(effects
@@
 			)
 		)
-		(property "Datasheet" "https://octopart.com/datasheet/16yxf100mefc6.3x11-rubycon-19941780"
+		(property "Datasheet" "https://octopart.com/datasheet/eeefth101xap-panasonic-19787188"
 			(at 55.88 200.66 0)
 			(effects
@@
 			)
 		)
-		(property "DigiKey PN" "1189-1856-ND"
+		(property "DigiKey PN" "PCE5024TR-ND"
 			(at 55.88 200.66 0)
 			(effects
@@
 			)
 		)
-		(property "LCSC Part #" " C338173"
+		(property "LCSC Part #" "C165974"
 			(at 55.88 200.66 0)
 			(effects
@@
 			)
 		)
-		(property "MPN" "16YXF100MEFC6.3X11"
+		(property "MPN" "EEEFTH101XAP"
 			(at 55.88 200.66 0)
 			(effects
@@
 			)
 		)
-		(property "Footprint" "Capacitor_THT:CP_Radial_D8.0mm_P2.50mm"
+		(property "Footprint" "Capacitor_SMD:CP_Elec_6.3x7.7"
 			(at 56.8452 140.97 0)
 			(effects
@@
 			)
 		)
-		(property "Datasheet" "https://octopart.com/datasheet/16yxf100mefc6.3x11-rubycon-19941780"
+		(property "Datasheet" "https://octopart.com/datasheet/eeefth101xap-panasonic-19787188"
 			(at 55.88 137.16 0)
 			(effects
@@
 			)
 		)
-		(property "DigiKey PN" "1189-1856-ND"
+		(property "DigiKey PN" "PCE5024TR-ND"
 			(at 55.88 137.16 0)
 			(effects
@@
 			)
 		)
-		(property "LCSC Part #" " C338173"
+		(property "LCSC Part #" "C165974"
 			(at 55.88 137.16 0)
 			(effects
@@
 			)
 		)
-		(property "MPN" "16YXF100MEFC6.3X11"
+		(property "MPN" "EEEFTH101XAP"
 			(at 55.88 137.16 0)
 			(effects
@@
 			)
 		)
-		(property "Footprint" "Capacitor_THT:CP_Radial_D8.0mm_P2.50mm"
+		(property "Footprint" "Capacitor_SMD:CP_Elec_6.3x7.7"
 			(at 177.4952 328.93 0)
 			(effects
@@
 			)
 		)
-		(property "Datasheet" "https://octopart.com/datasheet/16yxf100mefc6.3x11-rubycon-19941780"
+		(property "Datasheet" "https://octopart.com/datasheet/eeefth101xap-panasonic-19787188"
 			(at 176.53 325.12 0)
 			(effects
@@
 			)
 		)
-		(property "DigiKey PN" "1189-1856-ND"
+		(property "DigiKey PN" "PCE5024TR-ND"
 			(at 176.53 325.12 0)
 			(effects
@@
 			)
 		)
-		(property "LCSC Part #" " C338173"
+		(property "LCSC Part #" "C165974"
 			(at 176.53 325.12 0)
 			(effects
@@
 			)
 		)
-		(property "MPN" "16YXF100MEFC6.3X11"
+		(property "MPN" "EEEFTH101XAP"
 			(at 176.53 325.12 0)
 			(effects
@@
 			)
 		)
-		(property "Footprint" "Capacitor_THT:CP_Radial_D8.0mm_P2.50mm"
+		(property "Footprint" "Capacitor_SMD:CP_Elec_6.3x7.7"
 			(at 177.4952 81.28 0)
 			(effects
@@
 			)
 		)
-		(property "Datasheet" "https://octopart.com/datasheet/16yxf100mefc6.3x11-rubycon-19941780"
+		(property "Datasheet" "https://octopart.com/datasheet/eeefth101xap-panasonic-19787188"
 			(at 176.53 77.47 0)
 			(effects
@@
 			)
 		)
-		(property "DigiKey PN" "1189-1856-ND"
+		(property "DigiKey PN" "PCE5024TR-ND"
 			(at 176.53 77.47 0)
 			(effects
@@
 			)
 		)
-		(property "LCSC Part #" " C338173"
+		(property "LCSC Part #" "C165974"
 			(at 176.53 77.47 0)
 			(effects
@@
 			)
 		)
-		(property "MPN" "16YXF100MEFC6.3X11"
+		(property "MPN" "EEEFTH101XAP"
 			(at 176.53 77.47 0)
 			(effects
@@
 			)
 		)
-		(property "Footprint" "Capacitor_THT:CP_Radial_D8.0mm_P2.50mm"
+		(property "Footprint" "Capacitor_SMD:CP_Elec_6.3x7.7"
 			(at 177.4952 204.47 0)
 			(effects
@@
 			)
 		)
-		(property "Datasheet" "https://octopart.com/datasheet/16yxf100mefc6.3x11-rubycon-19941780"
+		(property "Datasheet" "https://octopart.com/datasheet/eeefth101xap-panasonic-19787188"
 			(at 176.53 200.66 0)
 			(effects
@@
 			)
 		)
-		(property "DigiKey PN" "1189-1856-ND"
+		(property "DigiKey PN" "PCE5024TR-ND"
 			(at 176.53 200.66 0)
 			(effects
@@
 			)
 		)
-		(property "LCSC Part #" " C338173"
+		(property "LCSC Part #" "C165974"
 			(at 176.53 200.66 0)
 			(effects
@@
 			)
 		)
-		(property "MPN" "16YXF100MEFC6.3X11"
+		(property "MPN" "EEEFTH101XAP"
 			(at 176.53 200.66 0)
 			(effects
@@
 			)
 		)
-		(property "Footprint" "Capacitor_THT:CP_Radial_D8.0mm_P2.50mm"
+		(property "Footprint" "Capacitor_SMD:CP_Elec_6.3x7.7"
 			(at 177.4952 140.97 0)
 			(effects
@@
 			)
 		)
-		(property "Datasheet" "https://octopart.com/datasheet/16yxf100mefc6.3x11-rubycon-19941780"
+		(property "Datasheet" "https://octopart.com/datasheet/eeefth101xap-panasonic-19787188"
 			(at 176.53 137.16 0)
 			(effects
@@
 			)
 		)
-		(property "DigiKey PN" "1189-1856-ND"
+		(property "DigiKey PN" "PCE5024TR-ND"
 			(at 176.53 137.16 0)
 			(effects
@@
 			)
 		)
-		(property "LCSC Part #" " C338173"
+		(property "LCSC Part #" "C165974"
 			(at 176.53 137.16 0)
 			(effects
@@
 			)
 		)
-		(property "MPN" "16YXF100MEFC6.3X11"
+		(property "MPN" "EEEFTH101XAP"
 			(at 176.53 137.16 0)
 			(effects
@@
 			)
 		)
-		(property "Footprint" "Capacitor_THT:CP_Radial_D8.0mm_P2.50mm"
+		(property "Footprint" "Capacitor_SMD:CP_Elec_6.3x7.7"
 			(at 56.8452 391.16 0)
 			(effects
@@
 			)
 		)
-		(property "Datasheet" "https://octopart.com/datasheet/16yxf100mefc6.3x11-rubycon-19941780"
+		(property "Datasheet" "https://octopart.com/datasheet/eeefth101xap-panasonic-19787188"
 			(at 55.88 387.35 0)
 			(effects
@@
 			)
 		)
-		(property "DigiKey PN" "1189-1856-ND"
+		(property "DigiKey PN" "PCE5024TR-ND"
 			(at 55.88 387.35 0)
 			(effects
@@
 			)
 		)
-		(property "LCSC Part #" " C338173"
+		(property "LCSC Part #" "C165974"
 			(at 55.88 387.35 0)
 			(effects
@@
 			)
 		)
-		(property "MPN" "16YXF100MEFC6.3X11"
+		(property "MPN" "EEEFTH101XAP"
 			(at 55.88 387.35 0)
 			(effects
@@
 			)
 		)
-		(property "Footprint" "Capacitor_THT:CP_Radial_D8.0mm_P2.50mm"
+		(property "Footprint" "Capacitor_SMD:CP_Elec_6.3x7.7"
 			(at 56.8452 266.7 0)
 			(effects
@@
 			)
 		)
-		(property "Datasheet" "https://octopart.com/datasheet/16yxf100mefc6.3x11-rubycon-19941780"
+		(property "Datasheet" "https://octopart.com/datasheet/eeefth101xap-panasonic-19787188"
 			(at 55.88 262.89 0)
 			(effects
@@
 			)
 		)
-		(property "DigiKey PN" "1189-1856-ND"
+		(property "DigiKey PN" "PCE5024TR-ND"
 			(at 55.88 262.89 0)
 			(effects
@@
 			)
 		)
-		(property "LCSC Part #" " C338173"
+		(property "LCSC Part #" "C165974"
 			(at 55.88 262.89 0)
 			(effects
@@
 			)
 		)
-		(property "MPN" "16YXF100MEFC6.3X11"
+		(property "MPN" "EEEFTH101XAP"
 			(at 55.88 262.89 0)
 			(effects
@@
 			)
 		)
-		(property "Footprint" "Capacitor_THT:CP_Radial_D8.0mm_P2.50mm"
+		(property "Footprint" "Capacitor_SMD:CP_Elec_6.3x7.7"
 			(at 177.4952 388.62 0)
 			(effects
@@
 			)
 		)
-		(property "Datasheet" "https://octopart.com/datasheet/16yxf100mefc6.3x11-rubycon-19941780"
+		(property "Datasheet" "https://octopart.com/datasheet/eeefth101xap-panasonic-19787188"
 			(at 176.53 384.81 0)
 			(effects
@@
 			)
 		)
-		(property "DigiKey PN" "1189-1856-ND"
+		(property "DigiKey PN" "PCE5024TR-ND"
 			(at 176.53 384.81 0)
 			(effects
@@
 			)
 		)
-		(property "LCSC Part #" " C338173"
+		(property "LCSC Part #" "C165974"
 			(at 176.53 384.81 0)
 			(effects
@@
 			)
 		)
-		(property "MPN" "16YXF100MEFC6.3X11"
+		(property "MPN" "EEEFTH101XAP"
 			(at 176.53 384.81 0)
 			(effects
@@
 			)
 		)
-		(property "Footprint" "Capacitor_THT:CP_Radial_D8.0mm_P2.50mm"
+		(property "Footprint" "Capacitor_SMD:CP_Elec_6.3x7.7"
 			(at 56.8452 328.93 0)
 			(effects
@@
 			)
 		)
-		(property "Datasheet" "https://octopart.com/datasheet/16yxf100mefc6.3x11-rubycon-19941780"
+		(property "Datasheet" "https://octopart.com/datasheet/eeefth101xap-panasonic-19787188"
 			(at 55.88 325.12 0)
 			(effects
@@
 			)
 		)
-		(property "DigiKey PN" "1189-1856-ND"
+		(property "DigiKey PN" "PCE5024TR-ND"
 			(at 55.88 325.12 0)
 			(effects
@@
 			)
 		)
-		(property "LCSC Part #" " C338173"
+		(property "LCSC Part #" "C165974"
 			(at 55.88 325.12 0)
 			(effects
@@
 			)
 		)
-		(property "MPN" "16YXF100MEFC6.3X11"
+		(property "MPN" "EEEFTH101XAP"
 			(at 55.88 325.12 0)
 			(effects
@@
 			)
 		)
-		(property "Footprint" "Capacitor_THT:CP_Radial_D8.0mm_P2.50mm"
+		(property "Footprint" "Capacitor_SMD:CP_Elec_6.3x7.7"
 			(at 177.4952 267.97 0)
 			(effects
@@
 			)
 		)
-		(property "Datasheet" "https://octopart.com/datasheet/16yxf100mefc6.3x11-rubycon-19941780"
+		(property "Datasheet" "https://octopart.com/datasheet/eeefth101xap-panasonic-19787188"
 			(at 176.53 264.16 0)
 			(effects
@@
 			)
 		)
-		(property "DigiKey PN" "1189-1856-ND"
+		(property "DigiKey PN" "PCE5024TR-ND"
 			(at 176.53 264.16 0)
 			(effects
@@
 			)
 		)
-		(property "LCSC Part #" " C338173"
+		(property "LCSC Part #" "C165974"
 			(at 176.53 264.16 0)
 			(effects
@@
 			)
 		)
-		(property "MPN" "16YXF100MEFC6.3X11"
+		(property "MPN" "EEEFTH101XAP"
 			(at 176.53 264.16 0)
 			(effects

Commit message: cleanup top, v0.4.2
Other:
- title: 12-12 Teensy G4.1 Arena Top Modular LED Display -> G4.1 Arena Top :: Modular LED Display
Changed lines of the file:
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@@
 	(paper "User" 304.8 508)
 	(title_block
-		(title "12-12 Teensy G4.1 Arena Top Modular LED Display")
-		(date "2025-07-22")
-		(rev "v0.4.1")
+		(title "G4.1 Arena Top :: Modular LED Display")
+		(date "2025-07-24")
+		(rev "v0.4.2")
 		(company "IORodeo for Reiserlab @ Janelia")
 	)
@@
 			(font
 				(size 5.08 5.08)
-				(thickness 0.508)
+				(thickness 1.016)
 				(bold yes)
 			)
