File: arena_12-12/arena_12-12_G4.1_top/power.kicad_sch (KiCad schematic)
At the start: 1 part, among them J4 Barrel_Jack

Commit message: bump version
Changed lines of the file:
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@@
 (kicad_sch
-	(version 20231120)
+	(version 20250114)
 	(generator "eeschema")
-	(generator_version "8.0")
+	(generator_version "9.0")
 	(paper "USLetter")
 	(title_block
 		(title "12-12 Teensy G4.1 Arena Top Modular LED Display")
-		(date "2024-12-23")
-		(rev "v0.3")
+		(date "2025-07-22")
+		(rev "v0.4")
 		(company "IORodeo for Reiserlab @ Janelia")
+	)
+	(text "Connection PCB top"
+		(exclude_from_sim no)
+		(at 105.664 75.184 0)
+		(effects
+			(font
+				(size 1.27 1.27)
+			)
+		)
+	)
+	(text "Power"
+		(exclude_from_sim no)
+		(at 115.189 21.082 0)
+		(effects
+			(font
+				(size 5.08 5.08)
+				(thickness 0.508)
+				(bold yes)
+			)
+			(justify left bottom)
+		)
 	)
 	(wire
@@
 		)
 	)
-	(text "Connection PCB top"
-		(exclude_from_sim no)
-		(at 105.664 75.184 0)
-		(effects
-			(font
-				(size 1.27 1.27)
-			)
-		)
-	)
-	(text "Power"
-		(exclude_from_sim no)
-		(at 115.189 21.082 0)
-		(effects
-			(font
-				(size 5.08 5.08)
-				(thickness 0.508)
-				(bold yes)
-			)
-			(justify left bottom)
-		)
-	)

Commit message: cleanup top, v0.4.2
Parts:
- J4: footprint arena_custom:DCJACK_2PIN_HIGHCURRENT -> Connector_BarrelJack:BarrelJack_CUI_PJ-036AH-SMT_Horizontal; symbol Connector:Barrel_Jack -> Connector:Barrel_Jack_Switch; DigiKey PN CP-063AH-ND -> CP-036AHPJTR-ND; LCSC Part # C2928097 -> C3094052; MPN PJ-063AH -> PJ-036AH-SMT-TR
Connections:
- no-connect marks 0 -> 1
Other:
- title: 12-12 Teensy G4.1 Arena Top Modular LED Display -> G4.1 Arena Top :: Modular LED Display
Changed lines of the file:
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@@
 	(paper "USLetter")
 	(title_block
-		(title "12-12 Teensy G4.1 Arena Top Modular LED Display")
-		(date "2025-07-22")
-		(rev "v0.4.1")
+		(title "G4.1 Arena Top :: Modular LED Display")
+		(date "2025-07-24")
+		(rev "v0.4.2")
 		(company "IORodeo for Reiserlab @ Janelia")
 	)
@@
 			(font
 				(size 5.08 5.08)
-				(thickness 0.508)
+				(thickness 1.016)
 				(bold yes)
 			)
@@
 		)
 	)
+	(no_connect
+		(at 92.71 82.55)
+	)
 	(wire
 		(pts
@@
 		(pts
 			(xy 196.85 45.72) (xy 196.85 50.8)
+		)
+		(stroke
+			(width 0)
+			(type default)
+		)
+	)
+	(wire
+		(pts
+			(xy 92.71 82.55) (xy 96.52 82.55)
 		)
 		(stroke
@@
 	)
 	(symbol
-		(lib_id "Connector:Barrel_Jack")
+		(lib_id "Connector:Barrel_Jack_Switch")
 		(at 104.14 82.55 0)
 		(mirror y)
@@
 		(fields_autoplaced yes)
 		(property "Reference" "J4"
-			(at 110.49 81.915 0)
+			(at 110.49 81.2799 0)
 			(effects
 				(font
@@
 		)
 		(property "Value" "Barrel_Jack"
-			(at 110.49 84.455 0)
+			(at 110.49 83.8199 0)
 			(effects
 				(font
@@
 			)
 		)
-		(property "Footprint" "arena_custom:DCJACK_2PIN_HIGHCURRENT"
+		(property "Footprint" "Connector_BarrelJack:BarrelJack_CUI_PJ-036AH-SMT_Horizontal"
 			(at 102.87 83.566 0)
 			(effects
@@
 			)
 		)
-		(property "Datasheet" "https://octopart.com/datasheet/pj-063ah-same+sky-106234056"
+		(property "Datasheet" "~"
 			(at 102.87 83.566 0)
 			(effects
@@
 			)
 		)
-		(property "Description" ""
+		(property "Description" "DC Barrel Jack with an internal switch"
 			(at 104.14 82.55 0)
 			(effects
@@
 			)
 		)
-		(property "DigiKey PN" "CP-063AH-ND"
+		(property "DigiKey PN" "CP-036AHPJTR-ND"
 			(at 104.14 82.55 0)
 			(effects
@@
 			)
 		)
-		(property "LCSC Part #" "C2928097"
+		(property "LCSC Part #" "C3094052"
 			(at 104.14 82.55 0)
 			(effects
@@
 			)
 		)
-		(property "MPN" "PJ-063AH"
+		(property "MPN" "PJ-036AH-SMT-TR"
 			(at 104.14 82.55 0)
 			(effects
@@
 		(pin "2"
 		)
-		(instances
+		(pin "3"
+		)
+		(instances
