File: arena_12-12/arena_12-12_v10_teensy/arena_12-12_v10_teensy.kicad_sch (KiCad schematic)
At the start: 0 parts

Commit message: add v10.3
Other:
- title: 12-12 Arena Teensy Modular LED Display -> Arena 12-12 Teensy Modular LED Display
Changed lines of the file:
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@@
 	(generator "eeschema")
 	(generator_version "9.0")
-	(paper "User" 279.4 203.2)
+	(paper "USLetter")
 	(title_block
-		(title "12-12 Arena Teensy Modular LED Display")
-		(date "2025-02-28")
-		(rev "v10.1")
+		(title "Arena 12-12 Teensy Modular LED Display")
+		(date "2024-12-23")
+		(rev "v10.3")
 		(company "IORodeo for Reiserlab @ Janelia")
 	)
@@
 			(project "arena_12-12_v10_teensy"
 				(path "/a2511654-3a17-43f1-8b9e-c45e375533dc"
-					(page "6")
+					(page "5")
 				)
 			)
@@
 			(project "arena_12-12_v10_teensy"
 				(path "/a2511654-3a17-43f1-8b9e-c45e375533dc"
-					(page "5")
-				)
-			)
+					(page "4")
+				)
+			)
